File: Carte Alimentation/carte_2015/carte_alim.kicad_pcb (KiCad board)
At the start: 2 copper layers, 102.9 x 70.5 mm, 58 parts, among them K1 CONN_3, P1 CONN_2, P10 CONN_2, P11 CONN_2, P12 CONN_2, P13 CONN_4, P2 CONN_2, P3 CONN_2, P4 CONN_5, P5 CONN_1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

Commit message: carte alim v2
Parts:
- U3, U4: value TL072 -> LM2903; footprint pin_array_4x2 -> Sockets_DIP:DIP-8__300
- moved D6 80.8 mm to (145.2, 203.2), turned to 270 degrees
- moved D9 76.2 mm to (145.2, 216.0), turned to 270 degrees
- moved D5 75.2 mm to (145.2, 209.8), turned to 90 degrees
- moved D8 73.5 mm to (145.2, 222.5), turned to 90 degrees
- moved 180u2 65.1 mm to (82.5, 221.0), turned to 180 degrees
- moved 5k4 61.9 mm to (140.0, 218.8), turned to 270 degrees
- moved 5k1 61.6 mm to (142.8, 191.0), turned to 90 degrees
- moved U3 60.6 mm to (128.5, 203.0), turned to 270 degrees
- moved D3 59.0 mm to (69.5, 175.0), turned to 0 degrees
- moved 5k2 58.2 mm to (136.5, 191.2), turned to 90 degrees
- moved 22u1 57.0 mm to (70.5, 221.0), turned to 270 degrees
- moved 5k3 55.1 mm to (135.8, 220.8), turned to 270 degrees
- moved C8 54.8 mm to (98.0, 208.8), turned to 180 degrees
- moved 180u1 51.3 mm to (93.0, 221.0)
- moved U4 51.0 mm to (121.5, 215.8), turned to 270 degrees
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Connections:
- P13 pad 3: (no net) -> Net-(P13-Pad3)
Routing:
- net GND: track 512.6 -> 630.6 mm
- net Net-(D8-Pad1): track 3.17 -> 85.3 mm
- net Net-(D5-Pad1): track 3.18 -> 74.7 mm
- net Net-(D3-Pad2): track 3.81 -> 69.4 mm
- net /alim_puissance_regul: track 110.3 -> 149.4 mm
- net Net-(F1-Pad1): track 21.0 -> 53.0 mm
- net Net-(100k2-Pad2): track 11.2 -> 41.5 mm
- net Net-(D10-Pad2): track 8.89 -> 34.8 mm
- net Net-(100k1-Pad2): track 12.5 -> 37.5 mm
- net Net-(D11-Pad2): track 9.42 -> 30.9 mm
- net Net-(D2-Pad2): track 3.81 -> 24.6 mm
- net Net-(D1-Pad1): track 21.7 -> 40.5 mm
- net Net-(5k2-Pad1): track 4.45 -> 22.8 mm
- net Net-(5k1-Pad1): track 4.45 -> 21.9 mm
- net Net-(D11-Pad1): track 40.2 -> 23.0 mm
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Other:
- board text added: "Carte Alim Robotronik© 2015 robin.moussu@gmail.com"
- board text removed: "Carte alim Robotronik© 2014 robin.moussu@gmail.com"

Commit message: plan de masse
Parts:
- moved R1 0.90 mm to (104.3, 174.3)
- moved R2 0.90 mm to (100.5, 174.3)
- moved R3 0.90 mm to (108.0, 174.3)
Routing:
- net GND: track 630.6 -> 626.8 mm
- net Net-(D3-Pad2): track 69.4 -> 68.1 mm
