File: Carte Alimentation/carte_2015/carte_alim.sch (KiCad schematic (older format))
At the start: 58 parts, among them K1 CONN_3, P1 CONN_2, P10 CONN_2, P11 CONN_2, P12 CONN_2, P13 CONN_4, P2 CONN_2, P3 CONN_2, P4 CONN_5, P5 CONN_1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

Commit message: carte alim v2
Parts:
- removed U3, U4: TL072, symbol TL072
- added U3, U4: LM2903, symbol LM2903
Changed lines of the file:
@@
 LIBS:valves
 LIBS:7905
-LIBS:carte_alim-cache
-EELAYER 27 0
+EELAYER 25 0
 EELAYER END
 $Descr A4 11693 8268
@@
 $EndComp
 $Comp
-L TL072 U3
-U 1 1 54DCC30A
-P 2200 5800
-F 0 "U3" H 2150 6000 60  0000 L CNN
-F 1 "TL072" H 2150 5550 60  0000 L CNN
-F 2 "" H 2200 5800 60  0000 C CNN
-F 3 "" H 2200 5800 60  0000 C CNN
-	1    2200 5800
-	1    0    0    -1
-$EndComp
-$Comp
-L TL072 U3
-U 2 1 54DCC319
-P 2200 6700
-F 0 "U3" H 2150 6900 60  0000 L CNN
-F 1 "TL072" H 2150 6450 60  0000 L CNN
-F 2 "" H 2200 6700 60  0000 C CNN
-F 3 "" H 2200 6700 60  0000 C CNN
-	2    2200 6700
-	1    0    0    -1
-$EndComp
-$Comp
 L LED D5
 U 1 1 54DCC332
@@
 $EndComp
 $Comp
-L TL072 U4
-U 1 1 54DCD1A7
-P 5400 5850
-F 0 "U4" H 5350 6050 60  0000 L CNN
-F 1 "TL072" H 5350 5600 60  0000 L CNN
-F 2 "" H 5400 5850 60  0000 C CNN
-F 3 "" H 5400 5850 60  0000 C CNN
-	1    5400 5850
-	1    0    0    -1
-$EndComp
-$Comp
-L TL072 U4
-U 2 1 54DCD1AD
-P 5400 6750
-F 0 "U4" H 5350 6950 60  0000 L CNN
-F 1 "TL072" H 5350 6500 60  0000 L CNN
-F 2 "" H 5400 6750 60  0000 C CNN
-F 3 "" H 5400 6750 60  0000 C CNN
-	2    5400 6750
-	1    0    0    -1
-$EndComp
-$Comp
 L LED D8
 U 1 1 54DCD1B3
@@
 Wire Wire Line
 	5150 2600 8000 2600
+$Comp
+L LM2903 U3
+U 1 1 550DC1BA
+P 2200 5800
+F 0 "U3" H 2350 5950 60  0000 C CNN
+F 1 "LM2903" H 2400 5600 60  0000 C CNN
+F 2 "" H 2200 5800 60  0000 C CNN
+F 3 "" H 2200 5800 60  0000 C CNN
+	1    2200 5800
+	1    0    0    -1
+$EndComp
+$Comp
+L LM2903 U3
+U 2 1 550DC27F
+P 2200 6700
+F 0 "U3" H 2350 6850 60  0000 C CNN
+F 1 "LM2903" H 2400 6500 60  0000 C CNN
+F 2 "" H 2200 6700 60  0000 C CNN
+F 3 "" H 2200 6700 60  0000 C CNN
+	2    2200 6700
+	1    0    0    -1
+$EndComp
+$Comp
+L LM2903 U4
+U 1 1 550DD3A9
+P 5400 5850
+F 0 "U4" H 5550 6000 60  0000 C CNN
+F 1 "LM2903" H 5600 5650 60  0000 C CNN
+F 2 "" H 5400 5850 60  0000 C CNN
+F 3 "" H 5400 5850 60  0000 C CNN
+	1    5400 5850
+	1    0    0    -1
+$EndComp
+$Comp
+L LM2903 U4
+U 2 1 550DD711
+P 5400 6750
+F 0 "U4" H 5550 6900 60  0000 C CNN
+F 1 "LM2903" H 5600 6550 60  0000 C CNN
+F 2 "" H 5400 6750 60  0000 C CNN
+F 3 "" H 5400 6750 60  0000 C CNN
+	2    5400 6750
+	1    0    0    -1
+$EndComp
 $EndSCHEMATC

Commit message: oubli sauvegarde
Parts:
- 0.01u1, 0.47u1, 22u1, C1, C3, C5, C6, C7, C8: footprint ~ -> Discret:C2
- 100k1, 100k2, 5k1, 5k2, 5k3, 5k4, R1, R2, R3, R4, R5, R6, R7: footprint ~ -> Discret:R4
- 15u1, 15u2, 15u3, 180u1, 180u2: footprint ~ -> Discret:CP4
- 5V1, D10, D11, D4, D7: footprint ~ -> Discret:D4
- D1, D2, D3, D5, D6, D8, D9: footprint ~ -> LEDs:LED-3MM
- F1, F2: footprint ~ -> Discret:FUSE5-20
- K1: footprint ~ -> PIN_ARRAY_3X1
- P1, P10, P11, P12, P13, P2, P3, P9: footprint ~ -> Connect:bornier2
- P4: footprint ~ -> Connect:bornier5
- P5, P6, P7, P8: footprint ~ -> PIN_ARRAY_1
- U3, U4: footprint (none) -> Sockets_DIP:DIP-8__300

Commit message: on avance
Parts:
- renumbered R4 to 1k, R6 to 1k, 100k2 to R254, 100k1 to R?
Other:
- moved on the sheet: D4, D7, R5, R7
