File: Carte Actionneurs-Capteurs/Carte Actionneurs-Capteurs.kicad_pcb (KiCad board)
At the start: 2 copper layers, 63 parts, among them K1 CONN_3, K10 CONN_3, K11 CONN_3, K12 CONN_3, K13 CONN_3, K14 CONN_3, K15 CONN_3, K16 CONN_3, K17 CONN_3, K18 CONN_3, K19 CONN_3, K2 CONN_3, K20 CONN_3, K21 CONN_3, K22 CONN_3, K23 CONN_3, K24 CONN_3, K25 CONN_3, K26 CONN_3, K27 CONN_3, K28 CONN_3, K29 CONN_3, K3 CONN_3, K4 CONN_3, K5 CONN_3, K6 CONN_3, K7 CONN_3, K8 CONN_3, K9 CONN_3, P1 CONN_1, P10 CONN_1, P11 CONN_1, P12 CONN_12, P13 CONN_12, P2 CONN_1, P3 CONN_2, P4 CONN_1, P5 CONN_1, P6 CONN_25X2, P8 CONN_1, P9 CONN_1

Commit message: fin routage
Parts:
- added R2: R, Discret:R3, F.Cu at (108.0, 94.5)
- added R23: R, Discret:R3, F.Cu at (108.0, 57.5)
- added R24: R, Discret:R3, F.Cu at (120.0, 84.0)
- moved P3 14.5 mm to (190.5, 135.5), turned to 270 degrees
- moved D1 10.5 mm to (190.5, 126.5), turned to 90 degrees
- moved R1 8.51 mm to (183.5, 134.5)
- moved R3 2.09 mm to (140.6, 57.1)
- moved R4 2.09 mm to (143.6, 57.1)
- moved R10 2.03 mm to (143.5, 74.7)
- moved R11 2.03 mm to (140.5, 80.7)
- moved R12 2.03 mm to (143.5, 80.7)
- moved R13 2.03 mm to (140.5, 86.7)
- moved R14 2.03 mm to (143.5, 86.7)
- moved R15 2.03 mm to (140.5, 92.7)
- moved R16 2.03 mm to (143.5, 92.7)
- moved R17 2.03 mm to (140.5, 98.7)
- moved R18 2.03 mm to (143.5, 98.7)
- moved R19 2.03 mm to (140.5, 104.7)
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Connections:
- D1 pad 1: PWR_IO_3 -> PWR_ADC_3
- K21 pad 2: PWR_IO_3 -> PWR_ADC_3
- K21 pad 3: PWR_ADC_4 -> PWR_IO_4
- K22 pad 2: PWR_IO_3 -> PWR_ADC_3
- K22 pad 3: PWR_ADC_4 -> PWR_IO_4
- K23 pad 2: PWR_IO_3 -> PWR_ADC_3
- K23 pad 3: PWR_ADC_4 -> PWR_IO_4
- K24 pad 2: PWR_IO_3 -> PWR_ADC_3
- K24 pad 3: PWR_ADC_4 -> PWR_IO_4
- K25 pad 2: PWR_IO_3 -> PWR_ADC_3
- K25 pad 3: PWR_ADC_4 -> PWR_IO_4
- K26 pad 2: PWR_IO_3 -> PWR_ADC_3
- K26 pad 3: PWR_ADC_4 -> PWR_IO_4
- K27 pad 2: PWR_IO_3 -> PWR_ADC_3
- K27 pad 3: PWR_ADC_4 -> PWR_IO_4
- K28 pad 2: PWR_IO_3 -> PWR_ADC_3
- K28 pad 3: PWR_ADC_4 -> PWR_IO_4
- K29 pad 2: PWR_IO_3 -> PWR_ADC_3
- K29 pad 3: PWR_ADC_4 -> PWR_IO_4
- P1 pad 1: PWR_IO_3 -> PWR_ADC_3
- P12 pad 10: PWR_IO_3 -> PWR_ADC_3
- P12 pad 2: PWR_ADC_4 -> PWR_IO_4
- P12 pad 3: PWR_IO_3 -> PWR_ADC_3
- P12 pad 4: PWR_ADC_4 -> PWR_ADC_3
- P12 pad 5: PWR_IO_3 -> PWR_IO_4
- P12 pad 7: PWR_ADC_4 -> PWR_IO_4
- P13 pad 10: PWR_IO_3 -> PWR_ADC_3
- P13 pad 2: PWR_ADC_4 -> PWR_IO_4
- P13 pad 3: PWR_IO_3 -> PWR_ADC_3
- P13 pad 4: PWR_ADC_4 -> PWR_ADC_3
- P13 pad 5: PWR_IO_3 -> PWR_IO_4
- P13 pad 7: PWR_ADC_4 -> PWR_IO_4
- P2 pad 1: PWR_IO_3 -> PWR_ADC_3
- P3 pad 1: PWR_IO_3 -> PWR_ADC_3
- P3 pad 2: PWR_ADC_4 -> PWR_IO_4
- P4 pad 1: PWR_ADC_4 -> PWR_IO_4
- P5 pad 1: PWR_ADC_4 -> PWR_IO_4
- P6 pad 1: PWR_ADC_4 -> PWR_IO_4
- P6 pad 10: PWR_ADC_4 -> PWR_IO_4
- P6 pad 12: PWR_ADC_4 -> PWR_IO_4
- P6 pad 2: PWR_ADC_4 -> PWR_IO_4
- P6 pad 23: PWR_ADC_4 -> PWR_IO_4
- P6 pad 25: PWR_ADC_4 -> PWR_IO_4
- P6 pad 38: PWR_ADC_4 -> PWR_IO_4
- P6 pad 4: PWR_ADC_4 -> PWR_IO_4
- P6 pad 40: PWR_ADC_4 -> PWR_IO_4
- P6 pad 42: PWR_ADC_4 -> PWR_IO_4
- P6 pad 44: PWR_ADC_4 -> PWR_IO_4
- P6 pad 46: PWR_ADC_4 -> PWR_IO_4
- P6 pad 48: PWR_ADC_4 -> PWR_IO_4
- P6 pad 49: PWR_ADC_4 -> PWR_IO_4
- P6 pad 50: PWR_ADC_4 -> PWR_IO_4
- P6 pad 6: PWR_ADC_4 -> PWR_IO_4
- P6 pad 8: PWR_ADC_4 -> PWR_IO_4
- R1 pad 1: PWR_ADC_4 -> PWR_IO_4
- R10 pad 1: PWR_ADC_4 -> PWR_IO_4
- R11 pad 1: PWR_IO_3 -> PWR_ADC_3
- R12 pad 1: PWR_ADC_4 -> PWR_IO_4
- R13 pad 1: PWR_IO_3 -> PWR_ADC_3
- R14 pad 1: PWR_ADC_4 -> PWR_IO_4
- R15 pad 1: PWR_IO_3 -> PWR_ADC_3
- R16 pad 1: PWR_ADC_4 -> PWR_IO_4
- R17 pad 1: PWR_IO_3 -> PWR_ADC_3
- R18 pad 1: PWR_ADC_4 -> PWR_IO_4
- R19 pad 1: PWR_IO_3 -> PWR_ADC_3
- R20 pad 1: PWR_ADC_4 -> PWR_IO_4
- R21 pad 1: PWR_IO_3 -> PWR_ADC_3
- R22 pad 1: PWR_ADC_4 -> PWR_IO_4
- R3 pad 1: PWR_IO_3 -> PWR_ADC_3
- R4 pad 1: PWR_ADC_4 -> PWR_IO_4
- R5 pad 1: PWR_IO_3 -> PWR_ADC_3
- R6 pad 1: PWR_ADC_4 -> PWR_IO_4
- R7 pad 1: PWR_IO_3 -> PWR_ADC_3
- R8 pad 1: PWR_ADC_4 -> PWR_IO_4
- R9 pad 1: PWR_IO_3 -> PWR_ADC_3
Routing:
- net PWR_IO_4: track 0.00 -> 872.5 mm
- net PWR_ADC_4: track 478.6 -> 0.00 mm
- net PWR_ADC_3: track 0.00 -> 399.5 mm
- net PWR_IO_3: track 298.2 -> 0.00 mm
- net PWR_IO_2: track 60.8 -> 115.9 mm
- net PWR_IO_1: track 60.6 -> 114.6 mm
- net IO6: track 103.2 -> 141.6 mm
- net IO8: track 89.9 -> 103.2 mm
- net IO10: track 77.0 -> 89.5 mm
- net IO9: track 83.2 -> 94.2 mm
- net IO4: track 116.4 -> 127.1 mm
- net IO7: track 96.5 -> 105.8 mm
- net IO3: track 123.1 -> 132.0 mm
- net IO2: track 129.7 -> 137.3 mm
- net IO11: track 127.8 -> 135.3 mm
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- added copper zone on B.Cu, net PWR_IO_4
- added copper zone on F.Cu, net PWR_IO_4
Other:
- board outline added: 108 x 102 mm
- board text added: "Carte Actionneurs Capteurs Robotronik 2014-2015"

Commit message: fini carte actionneurs-capteurs
Parts:
- moved R1 0.28 mm to (183.6, 134.2)
Routing:
- net PWR_IO_4: track 872.5 -> 857.5 mm
- net Net-(D1-Pad2): track 9.68 -> 9.08 mm

Commit message: réparation carte actionneurs-capteurs
Parts:
- K1, K10, K11, K12, K13, K14, K15, K16, K17, K18, K19, K2, K20, K21, K22, K23, K24, K25, K26, K27, K28, K29, K3, K4, K5, K6, K7, K8, K9: value CONN_3 -> CONN_01x03
Connections:
- net PWR_IO_4 renamed PWR_ADC_4
Routing:
- added copper zone on B.Cu, net PWR_IO_4
- added copper zone on F.Cu, net PWR_IO_4
- removed copper zone on B.Cu, net PWR_ADC_4
- removed copper zone on F.Cu, net PWR_ADC_4
