File: Carte Actionneurs-Capteurs mini/Carte Actionneurs-Capteurs.kicad_pcb (KiCad board)
At the start: 2 copper layers, 46.5 x 102 mm, 38 parts, among them K1 CONN_3, K11 CONN_3, K12 CONN_3, K13 CONN_3, K14 CONN_3, K15 CONN_3, K2 CONN_3, K21 CONN_3, K22 CONN_3, K23 CONN_3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

Commit message: réparation carte actionneurs capteurs mini
Parts:
- K1, K11, K12, K13, K14, K15, K2, K21, K22, K23, K24, K25, K26, K3, K4, K5: value CONN_3 -> CONN_01X03
Connections:
- net PWR_IO_4 renamed PWR_ADC_4
Routing:
- added copper zone on B.Cu, net PWR_IO_4
- added copper zone on F.Cu, net PWR_IO_4
- removed copper zone on B.Cu, net PWR_ADC_4
- removed copper zone on F.Cu, net PWR_ADC_4
