File: Carte Alimentation/AlimDetect/AlimDetect_4c.sch (KiCad schematic (older format))
At the start: 18 parts, among them P1 CONN_2, P2 CONN_2, P3 CONN_2, U1 LM2678

Commit message: Circuit de détection du niveau des batteries
Parts:
- removed P?: CONN_5, ~, symbol CONN_5
- added D?: ZENER, ~, symbol ZENER
- added D? (x4): LED, ~, symbol LED
- added P?: CONN_5, ~, symbol CONN_5
- added R? (x26): R, ~, symbol R
- added U? (x8): TLC274, symbol TLC274
- added U? (x4): 74HCT00, ~, symbol 74HCT00
- added U?: KMIG1240, ~, symbol KMIG1240
- added U?: 7805, ~, symbol 7805
Connections:
- net labels added: +5V, Vref
- wire segments 29 -> 130

Commit message: Regul 5V à la bonne place
Connections:
- wire segments 130 -> 129

Commit message: Annotation de AlimDetect_4c.sch
Parts:
- gave numbers to parts that had none: 37

Commit message: Condensateurs de découplage sur AlimDetect_4c.sch
Parts:
- added C10, C8, C9: C, ~, symbol C
Connections:
- wire segments 129 -> 131
Other:
- note added: "IN_DETECT"

Commit message: Correction logique de détection du niveau des batteries
Parts:
- removed R27: R, ~, symbol R
- removed U5: 74HCT00, ~, symbol 74HCT00
- added R?: R, ~, symbol R
- added U? (x4): 74LS08, ~, symbol 74LS08
Connections:
- wire segments 131 -> 130
- no-connect marks 1 -> 4

Commit message: ERC ok pour 2 et 4 celulles
Parts:
- gave numbers to parts that had none: 2

Commit message: Réparation de 4c.sch et 2c.sch
Parts:
- removed P1, P2, P3: CONN_2, ~, symbol CONN_2
- removed P4: CONN_5, ~, symbol CONN_5
- added P? (x3): CONN_01X02, symbol CONN_01X02
- added P?: CONN_01X05, symbol CONN_01X05
Connections:
- wire segments 130 -> 175

Commit message: Correction logique de détection
Parts:
- gave numbers to parts that had none: 4
