File: Carte Alimentation/AlimDetect/AlimDetect_2c.sch (KiCad schematic (older format))
At the start: 29 parts, among them K1 CONN_3, P1 CONN_2, P2 CONN_2, P3 CONN_2, U1 7805, U2 TLC274, U3 74LS08, U4 KMIG1240

Commit message: ERC ok pour 2 et 4 celulles
Parts:
- added C1, C2, C3, C4: C, ~, symbol C
- added U5: 7805, ~, symbol 7805
Connections:
- wire segments 64 -> 72

Commit message: réparé alimDetect 2C
Parts:
- D2: symbol DIODE -> D
- K1: value CONN_3 -> CONN_01X03; symbol CONN_3 -> CONN_01X03
- P1, P2, P3: value CONN_2 -> CONN_01X02; symbol CONN_2 -> CONN_01X02
Connections:
- wire segments 72 -> 71

Commit message: Réparation de 4c.sch et 2c.sch
Changed lines of the file:
@@
 LIBS:valves
 LIBS:kmig1240
+LIBS:AlimDetect_2c-cache
 EELAYER 25 0
 EELAYER END
@@
 F 3 "~" H 1500 1250 60  0000 C CNN
 	1    1500 1250
-	-1   0    0    -1
+	-1   0    0    1
 $EndComp
 $Comp
@@
 F 3 "~" H 2900 1200 60  0000 C CNN
 	1    2900 1200
-	1    0    0    -1
+	-1   0    0    -1
 $EndComp
 $Comp
@@
 F 3 "~" H 6050 1250 60  0000 C CNN
 	1    6050 1250
-	1    0    0    -1
+	1    0    0    1
 $EndComp
 $Comp
@@
 F 3 "~" H 6050 2250 60  0000 C CNN
 	1    6050 2250
-	1    0    0    -1
+	1    0    0    1
 $EndComp
 $Comp
@@
 L GND #PWR013
 U 1 1 568EA93A
-P 650 4150
-F 0 "#PWR013" H 650 4150 30  0001 C CNN
-F 1 "GND" H 650 4080 30  0001 C CNN
-F 2 "" H 650 4150 60  0000 C CNN
-F 3 "" H 650 4150 60  0000 C CNN
-	1    650  4150
+P 1000 5850
+F 0 "#PWR013" H 1000 5850 30  0001 C CNN
+F 1 "GND" H 1000 5780 30  0001 C CNN
+F 2 "" H 1000 5850 60  0000 C CNN
+F 3 "" H 1000 5850 60  0000 C CNN
+	1    1000 5850
 	1    0    0    -1
 $EndComp
@@
 F 3 "~" H 9600 6000 60  0000 C CNN
 	1    9600 6000
-	0    -1   -1   0
+	0    -1   1    0
 $EndComp
 $Comp
@@
 F 3 "~" H 6550 3900 60  0000 C CNN
 	1    6550 3900
-	1    0    0    -1
+	-1   0    0    -1
 $EndComp
 $Comp
@@
 F 3 "~" H 6550 5100 60  0000 C CNN
 	1    6550 5100
-	1    0    0    -1
+	-1   0    0    -1
 $EndComp
 $Comp
@@
 L PWR_FLAG #FLG025
 U 1 1 568EAA0B
-P 650 3900
-F 0 "#FLG025" H 650 3995 30  0001 C CNN
-F 1 "PWR_FLAG" H 650 4080 30  0000 C CNN
-F 2 "" H 650 3900 60  0000 C CNN
-F 3 "" H 650 3900 60  0000 C CNN
-	1    650  3900
+P 700 5650
+F 0 "#FLG025" H 700 5745 30  0001 C CNN
+F 1 "PWR_FLAG" H 700 5830 30  0000 C CNN
+F 2 "" H 700 5650 60  0000 C CNN
+F 3 "" H 700 5650 60  0000 C CNN
+	1    700  5650
 	1    0    0    -1
 $EndComp
@@
 L 7805 U1
 U 1 1 568EAA11
-P 1500 6700
-F 0 "U1" H 1650 6504 60  0000 C CNN
-F 1 "7805" H 1500 6900 60  0000 C CNN
-F 2 "~" H 1500 6700 60  0000 C CNN
-F 3 "~" H 1500 6700 60  0000 C CNN
-	1    1500 6700
+P 1400 3150
+F 0 "U1" H 1550 2954 60  0000 C CNN
+F 1 "7805" H 1400 3350 60  0000 C CNN
+F 2 "~" H 1400 3150 60  0000 C CNN
+F 3 "~" H 1400 3150 60  0000 C CNN
+	1    1400 3150
 	1    0    0    -1
 $EndComp
@@
 L GND #PWR027
 U 1 1 568EAF33
-P 1500 6950
-F 0 "#PWR027" H 1500 6950 30  0001 C CNN
-F 1 "GND" H 1500 6880 30  0001 C CNN
-F 2 "" H 1500 6950 60  0000 C CNN
-F 3 "" H 1500 6950 60  0000 C CNN
-	1    1500 6950
+P 1400 3400
+F 0 "#PWR027" H 1400 3400 30  0001 C CNN
+F 1 "GND" H 1400 3330 30  0001 C CNN
+F 2 "" H 1400 3400 60  0000 C CNN
+F 3 "" H 1400 3400 60  0000 C CNN
+	1    1400 3400
 	1    0    0    -1
 $EndComp
@@
 L +5V #PWR028
 U 1 1 568EAF42
-P 2000 6450
-F 0 "#PWR028" H 2000 6540 20  0001 C CNN
-F 1 "+5V" H 2000 6540 30  0000 C CNN
-F 2 "" H 2000 6450 60  0000 C CNN
-F 3 "" H 2000 6450 60  0000 C CNN
-	1    2000 6450
+P 1900 2900
+F 0 "#PWR028" H 1900 2990 20  0001 C CNN
+F 1 "+5V" H 1900 2990 30  0000 C CNN
+F 2 "" H 1900 2900 60  0000 C CNN
+F 3 "" H 1900 2900 60  0000 C CNN
+	1    1900 2900
 	1    0    0    -1
 $EndComp
@@
 Connection ~ 1000 3900
 Wire Wire Line
-	650  3900 650  4150
-Wire Wire Line
-	650  3900 3100 3900
-Connection ~ 1300 5100
-Wire Wire Line
 	1300 4100 3100 4100
 Wire Wire Line
@@
 Connection ~ 1800 1200
 Wire Wire Line
-	1000 4600 1000 3900
+	1000 3100 1000 4600
 Wire Wire Line
 	1000 4700 1300 4700
@@
 	1300 4100 1300 5100
 Connection ~ 1300 4700
-Wire Wire Line
-	1000 4800 1000 6650
-Wire Wire Line
-	1000 6650 1100 6650
 Connection ~ 1000 5300
 Wire Wire Line
-	1900 6650 2000 6650
-Wire Wire Line
-	2000 6650 2000 6450
+	1800 3100 1900 3100
+Wire Wire Line
+	1900 3100 1900 2900
 Wire Wire Line
 	4900 3800 4000 3800
@@
 Wire Wire Line
 	3400 3400 3550 3400
+Wire Wire Line
+	1000 4800 1000 5850
+Wire Wire Line
+	1000 3900 3100 3900
+Wire Wire Line
+	700  5650 700  5700
+Wire Wire Line
+	700  5700 1000 5700
+Connection ~ 1000 5700
 $EndSCHEMATC

Commit message: Correction logique de détection
Parts:
- added C? (x2): C, symbol C
Connections:
- wire segments 71 -> 78
Changed lines of the file:
@@
 L +5V #PWR05
 U 1 1 568EA8CE
+P 2250 5500
+F 0 "#PWR05" H 2250 5590 20  0001 C CNN
+F 1 "+5V" H 2250 5590 30  0000 C CNN
+F 2 "" H 2250 5500 60  0000 C CNN
+F 3 "" H 2250 5500 60  0000 C CNN
+	1    2250 5500
+	1    0    0    1
+$EndComp
+$Comp
+L GND #PWR06
+U 1 1 568EA8D4
 P 2250 4900
-F 0 "#PWR05" H 2250 4990 20  0001 C CNN
-F 1 "+5V" H 2250 4990 30  0000 C CNN
+F 0 "#PWR06" H 2250 4900 30  0001 C CNN
+F 1 "GND" H 2250 4830 30  0001 C CNN
 F 2 "" H 2250 4900 60  0000 C CNN
 F 3 "" H 2250 4900 60  0000 C CNN
 	1    2250 4900
-	1    0    0    -1
-$EndComp
-$Comp
-L GND #PWR06
-U 1 1 568EA8D4
-P 2250 5500
-F 0 "#PWR06" H 2250 5500 30  0001 C CNN
-F 1 "GND" H 2250 5430 30  0001 C CNN
-F 2 "" H 2250 5500 60  0000 C CNN
-F 3 "" H 2250 5500 60  0000 C CNN
-	1    2250 5500
-	1    0    0    -1
+	1    0    0    1
 $EndComp
 $Comp
@@
 F 3 "" H 3700 4000 60  0000 C CNN
 	2    3700 4000
-	1    0    0    -1
+	1    0    0    1
 $EndComp
 $Comp
@@
 L +5V #PWR08
 U 1 1 568EA8FE
+P 3600 4300
+F 0 "#PWR08" H 3600 4390 20  0001 C CNN
+F 1 "+5V" H 3600 4390 30  0000 C CNN
+F 2 "" H 3600 4300 60  0000 C CNN
+F 3 "" H 3600 4300 60  0000 C CNN
+	1    3600 4300
+	1    0    0    1
+$EndComp
+$Comp
+L GND #PWR09
+U 1 1 568EA904
 P 3600 3700
-F 0 "#PWR08" H 3600 3790 20  0001 C CNN
-F 1 "+5V" H 3600 3790 30  0000 C CNN
+F 0 "#PWR09" H 3600 3700 30  0001 C CNN
+F 1 "GND" H 3600 3630 30  0001 C CNN
 F 2 "" H 3600 3700 60  0000 C CNN
 F 3 "" H 3600 3700 60  0000 C CNN
 	1    3600 3700
-	1    0    0    -1
-$EndComp
-$Comp
-L GND #PWR09
-U 1 1 568EA904
-P 3600 4300
-F 0 "#PWR09" H 3600 4300 30  0001 C CNN
-F 1 "GND" H 3600 4230 30  0001 C CNN
-F 2 "" H 3600 4300 60  0000 C CNN
-F 3 "" H 3600 4300 60  0000 C CNN
-	1    3600 4300
-	1    0    0    -1
+	1    0    0    1
 $EndComp
 $Comp
@@
 L GND #PWR013
 U 1 1 568EA93A
-P 1000 5850
-F 0 "#PWR013" H 1000 5850 30  0001 C CNN
-F 1 "GND" H 1000 5780 30  0001 C CNN
-F 2 "" H 1000 5850 60  0000 C CNN
-F 3 "" H 1000 5850 60  0000 C CNN
-	1    1000 5850
+P 1350 3550
+F 0 "#PWR013" H 1350 3550 30  0001 C CNN
+F 1 "GND" H 1350 3480 30  0001 C CNN
+F 2 "" H 1350 3550 60  0000 C CNN
+F 3 "" H 1350 3550 60  0000 C CNN
+	1    1350 3550
 	1    0    0    -1
 $EndComp
@@
 F 3 "" H 2350 5200 60  0000 C CNN
 	1    2350 5200
-	1    0    0    -1
+	1    0    0    1
 $EndComp
 $Comp
@@
 L PWR_FLAG #FLG025
 U 1 1 568EAA0B
-P 700 5650
-F 0 "#FLG025" H 700 5745 30  0001 C CNN
-F 1 "PWR_FLAG" H 700 5830 30  0000 C CNN
-F 2 "" H 700 5650 60  0000 C CNN
-F 3 "" H 700 5650 60  0000 C CNN
-	1    700  5650
+P 700 3400
+F 0 "#FLG025" H 700 3495 30  0001 C CNN
+F 1 "PWR_FLAG" H 700 3580 30  0000 C CNN
+F 2 "" H 700 3400 60  0000 C CNN
+F 3 "" H 700 3400 60  0000 C CNN
+	1    700  3400
 	1    0    0    -1
 $EndComp
@@
 L 7805 U1
 U 1 1 568EAA11
-P 1400 3150
-F 0 "U1" H 1550 2954 60  0000 C CNN
-F 1 "7805" H 1400 3350 60  0000 C CNN
-F 2 "~" H 1400 3150 60  0000 C CNN
-F 3 "~" H 1400 3150 60  0000 C CNN
-	1    1400 3150
+P 1550 6700
+F 0 "U1" H 1700 6504 60  0000 C CNN
+F 1 "7805" H 1550 6900 60  0000 C CNN
+F 2 "~" H 1550 6700 60  0000 C CNN
+F 3 "~" H 1550 6700 60  0000 C CNN
+	1    1550 6700
 	1    0    0    -1
 $EndComp
@@
 F 3 "~" H 800 4700 60  0000 C CNN
 	1    800  4700
-	-1   0    0    1
-$EndComp
-$Comp
-L GND #PWR027
-U 1 1 568EAF33
-P 1400 3400
-F 0 "#PWR027" H 1400 3400 30  0001 C CNN
-F 1 "GND" H 1400 3330 30  0001 C CNN
-F 2 "" H 1400 3400 60  0000 C CNN
-F 3 "" H 1400 3400 60  0000 C CNN
-	1    1400 3400
-	1    0    0    -1
+	-1   0    0    -1
 $EndComp
 $Comp
 L +5V #PWR028
 U 1 1 568EAF42
-P 1900 2900
-F 0 "#PWR028" H 1900 2990 20  0001 C CNN
-F 1 "+5V" H 1900 2990 30  0000 C CNN
-F 2 "" H 1900 2900 60  0000 C CNN
-F 3 "" H 1900 2900 60  0000 C CNN
-	1    1900 2900
+P 2050 6450
+F 0 "#PWR028" H 2050 6540 20  0001 C CNN
+F 1 "+5V" H 2050 6540 30  0000 C CNN
+F 2 "" H 2050 6450 60  0000 C CNN
+F 3 "" H 2050 6450 60  0000 C CNN
+	1    2050 6450
 	1    0    0    -1
 $EndComp
@@
 Connection ~ 1800 1200
 Wire Wire Line
-	1000 3100 1000 4600
-Wire Wire Line
 	1000 4700 1300 4700
 Wire Wire Line
@@
 Connection ~ 1000 5300
 Wire Wire Line
-	1800 3100 1900 3100
-Wire Wire Line
-	1900 3100 1900 2900
+	1950 6650 2050 6650
+Wire Wire Line
+	2050 6450 2050 6700
 Wire Wire Line
 	4900 3800 4000 3800
@@
 	3400 3400 3550 3400
 Wire Wire Line
-	1000 4800 1000 5850
-Wire Wire Line
 	1000 3900 3100 3900
 Wire Wire Line
-	700  5650 700  5700
-Wire Wire Line
-	700  5700 1000 5700
-Connection ~ 1000 5700
+	700  3400 700  3450
+Wire Wire Line
+	700  3450 1350 3450
+Connection ~ 1000 3450
+Wire Wire Line
+	5100 4300 5100 4200
+Wire Wire Line
+	1000 3450 1000 4600
+Wire Wire Line
+	1000 4800 1000 6700
+Wire Wire Line
+	1350 3450 1350 3550
+Wire Wire Line
+	5100 3600 5100 3500
+Wire Wire Line
+	1000 6650 1150 6650
+$Comp
+L C C?
+U 1 1 56A29008
+P 1000 6850
+F 0 "C?" H 1025 6950 50  0000 L CNN
+F 1 "C" H 1025 6750 50  0000 L CNN
+F 2 "" H 1038 6700 50  0000 C CNN
+F 3 "" H 1000 6850 50  0000 C CNN
+	1    1000 6850
+	1    0    0    -1
+$EndComp
+$Comp
+L C C?
+U 1 1 56A290DA
+P 2050 6850
+F 0 "C?" H 2075 6950 50  0000 L CNN
+F 1 "C" H 2075 6750 50  0000 L CNN
+F 2 "" H 2088 6700 50  0000 C CNN
+F 3 "" H 2050 6850 50  0000 C CNN
+	1    2050 6850
+	1    0    0    -1
+$EndComp
+$Comp
+L GND #PWR?
+U 1 1 56A29168
+P 2050 7100
+F 0 "#PWR?" H 2050 6850 50  0001 C CNN
+F 1 "GND" H 2050 6950 50  0000 C CNN
+F 2 "" H 2050 7100 50  0000 C CNN
+F 3 "" H 2050 7100 50  0000 C CNN
+	1    2050 7100
+	1    0    0    -1
+$EndComp
+$Comp
+L GND #PWR?
+U 1 1 56A291F8
+P 1000 7100
+F 0 "#PWR?" H 1000 6850 50  0001 C CNN
+F 1 "GND" H 1000 6950 50  0000 C CNN
+F 2 "" H 1000 7100 50  0000 C CNN
+F 3 "" H 1000 7100 50  0000 C CNN
+	1    1000 7100
+	1    0    0    -1
+$EndComp
+$Comp
+L GND #PWR?
+U 1 1 56A29281
+P 1550 7100
+F 0 "#PWR?" H 1550 7100 30  0001 C CNN
+F 1 "GND" H 1550 7030 30  0001 C CNN
+F 2 "" H 1550 7100 60  0000 C CNN
+F 3 "" H 1550 7100 60  0000 C CNN
+	1    1550 7100
+	1    0    0    -1
+$EndComp
+Connection ~ 2050 6650
+Wire Wire Line
+	2050 7000 2050 7100
+Wire Wire Line
+	1550 7100 1550 6950
+Wire Wire Line
+	1000 7100 1000 7000
+Connection ~ 1000 6650
 $EndSCHEMATC

Commit message: Ajustement avant réalisation des PCB par Pisa
Parts:
- removed C2: C, ~, symbol C
- removed C? (x2): C, symbol C
- removed U1: 7805, ~, symbol 7805
- removed U2: TLC274, symbol TLC274
- added D6: LED, LEDs:LED-3MM, symbol LED
- added P4: CONN_01X02, Pin_Headers:Pin_Header_Straight_1x02, symbol CONN_01X02
- added R16, R17: 250, Resistors_SMD:R_0603_HandSoldering, symbol R
- added U1: TLC274, Housings_SOIC:SOIC-14_3.9x8.7mm_Pitch1.27mm, symbol TLC274
- C1: value C -> 0.33µ; footprint ~ -> Capacitors_SMD:C_0603_HandSoldering
- C3: value C -> 0.1µ; footprint ~ -> Capacitors_SMD:C_0603_HandSoldering
- C4: footprint ~ -> Capacitors_ThroughHole:C_Radial_D18_L36_P7.5
- D1: footprint ~ -> LEDs:LED-3MM
- D2: value DIODE -> 1N5404; footprint ~ -> Diodes_ThroughHole:Diode_DO-201AD_Horizontal_RM15
- D3, D4: footprint ~ -> LEDs:LED_0603
- D5: footprint ~ -> Discret:D3
- F1: footprint ~ -> Fuse_Holders_and_Fuses:Fuseholder5x20_horiz_open_inline_Type-I
- K1: footprint ~ -> Pin_Headers:Pin_Header_Angled_1x03
- P1, P2, P3: footprint ~ -> Connect:bornier2
- R1, R2, R3, R5, R6, R7, R8, R9: footprint ~ -> Resistors_SMD:R_0603_HandSoldering
- R10, R11: value R -> 15k; footprint ~ -> Resistors_SMD:R_0603_HandSoldering
- R12, R13: value R -> 150; footprint ~ -> Resistors_SMD:R_0603_HandSoldering
- R14: value R -> 82; footprint ~ -> Resistors_SMD:R_0603_HandSoldering
- R15: value R -> 380; footprint ~ -> Resistors_ThroughHole:Resistor_Horizontal_RM10mm
- R4: value R -> 820; footprint ~ -> Resistors_ThroughHole:Resistor_Horizontal_RM10mm
- U3: footprint ~ -> Housings_SOIC:SOIC-14_3.9x8.7mm_Pitch1.27mm
- U4: footprint ~ -> buzz:kmig1240
- U5: footprint ~ -> TO_SOT_Packages_THT:TO-220_Neutral123_Horizontal; symbol 7805 -> 7805-RESCUE-AlimDetect_2c
Connections:
- net labels added: elec_redressé
- no-connect marks 9 -> 3
Other:
- note added: "ELEC_REGUL_5V\n"
- note removed: "ELEC"
- note removed: "ELEC_REGUL"
