File: Carte Alimentation/AlimDetect/AlimDetect_4c.kicad_pcb (KiCad board)
At the start: 2 copper layers, 56 parts, among them P1 CONN_01X05, P2 CONN_01X02, P3 CONN_01X02, P4 CONN_01X02, U1 LM2678, U2 7805, U3 TLC274, U4 TLC274, U5 74LS08, U6 KMIG1240

Commit message: Ajout cavalier buzzer et plans de masse 4c
Parts:
- added P5: CONN_01X02, Pin_Headers:Pin_Header_Straight_1x02, F.Cu at (131.4, 69.2)
- moved P3 3.18 mm to (135.9, 57.8)
- moved P4 3.18 mm to (135.9, 41.3)
- moved U6 1.91 mm to (131.4, 98.4)
Connections:
- U5 pad 11: Net-(U5-Pad11) -> Net-(P5-Pad2)
- U6 pad 2: Net-(U5-Pad11) -> Net-(P5-Pad1)
Routing:
- net Net-(P5-Pad1): track 0.00 -> 40.8 mm, vias 0 -> 1
- net Net-(P5-Pad2): track 0.00 -> 37.9 mm, vias 0 -> 1
- net Net-(U5-Pad11): track 22.5 -> 0.00 mm
- net +5V: track 74.0 -> 84.6 mm, vias 3 -> 4
- net /PWR_redressé: track 276.2 -> 273.1 mm
- net Net-(C6-Pad1): track 69.9 -> 66.8 mm
- net GND: track 633.4 -> 632.9 mm
- added copper zone on B.Cu, net GND
- added copper zone on F.Cu, net GND

Commit message: Ajustement avant réalisation des PCB par Pisa
Parts:
- added C4: 100n, Capacitors_SMD:C_0603_HandSoldering, F.Cu at (83.8, 125.7)
- added C7: 100n, Capacitors_SMD:C_0603_HandSoldering, F.Cu at (121.9, 118.1)
- added R28: 510, Resistors_SMD:R_0603_HandSoldering, F.Cu at (91.4, 134.6)
- added R29: 510, Resistors_SMD:R_0603_HandSoldering, F.Cu at (103.5, 135.9)
- added R30: 510, Resistors_ThroughHole:Resistor_Horizontal_RM7mm, F.Cu at (102.9, 107.3)
- added R31: 510, Resistors_SMD:R_0603_HandSoldering, F.Cu at (103.5, 118.1)
- U2: value 7805 -> 7805_correctPin
- moved D9 44.2 mm to (62.2, 104.1), turned to 180 degrees
- moved C1 42.3 mm to (80.0, 88.9)
- moved C2 42.3 mm to (64.1, 88.9)
- moved C8 42.3 mm to (142.9, 106.7)
- moved C9 42.3 mm to (142.9, 111.8)
- moved D2 42.3 mm to (88.9, 81.9)
- moved R1 42.3 mm to (88.9, 64.8)
- moved R10 42.3 mm to (91.4, 122.6)
- moved R24 42.3 mm to (112.4, 106.7)
- moved R7 42.3 mm to (71.1, 121.3)
- moved C6 42.3 mm to (117.5, 90.8)
- moved P2 42.3 mm to (52.1, 74.9)
- moved P4 42.3 mm to (167.6, 69.2)
- moved C10 42.3 mm to (111.8, 66.7)
- moved C3 42.3 mm to (100.3, 93.3)
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Connections:
- D9 pad 1: GND -> Net-(D9-Pad1)
- D9 pad 2: Net-(D9-Pad2) -> GND
- R27 pad 2: Net-(D9-Pad2) -> Net-(D9-Pad1)
- R8 pad 2: Net-(R8-Pad2) -> Net-(R28-Pad2)
- R9 pad 2: Net-(R9-Pad2) -> Net-(R29-Pad2)
- U3 pad 1: Net-(R8-Pad2) -> Net-(R28-Pad2)
- U3 pad 7: Net-(R9-Pad2) -> Net-(R29-Pad2)
- U4 pad 10: Net-(R16-Pad2) -> Net-(R31-Pad1)
- U4 pad 12: Net-(R17-Pad2) -> Net-(R30-Pad1)
- U4 pad 3: Net-(R8-Pad2) -> Net-(R28-Pad1)
- U4 pad 5: Net-(R9-Pad2) -> Net-(R29-Pad1)
Routing:
- net Net-(R8-Pad2): track 85.6 -> 0.00 mm, vias 2 -> 0
- net Net-(R9-Pad2): track 59.7 -> 0.00 mm, vias 4 -> 0
- net Net-(R28-Pad2): track 0.00 -> 51.2 mm
- net Net-(R29-Pad2): track 0.00 -> 36.0 mm, vias 0 -> 2
- net Net-(R16-Pad2): track 69.0 -> 33.0 mm, vias 4 -> 2
- net Net-(R31-Pad1): track 0.00 -> 35.0 mm, vias 0 -> 2
- net Net-(R28-Pad1): track 0.00 -> 32.1 mm, vias 0 -> 2
- net Net-(R29-Pad1): track 0.00 -> 22.8 mm, vias 0 -> 2
- net Net-(R17-Pad2): track 34.1 -> 12.9 mm, vias 2 -> 1
- net /PWR_redressé: track 273.1 -> 291.1 mm
- net Net-(R30-Pad1): track 0.00 -> 15.6 mm, vias 0 -> 1
- net Net-(D9-Pad1): track 0.00 -> 10.1 mm
- net Net-(D9-Pad2): track 10.1 -> 0.00 mm
- net Net-(R18-Pad1): track 38.7 -> 45.0 mm
- net GND: track 632.9 -> 629.7 mm
Other:
- net class Default: via_dia 0.6 -> 0.9; via_drill 0.4 -> 0.8
- board text added: "1"
- board text added: "2"
- board text added: "3"
- board text added: "4"
- board text added: "4/02/2016 Carte Alim 4c - Robotronik Alexis"
- board text added: "Connect"
- board text added: "NON_REGUL"
- board text added: "REGUL"
- board text added: "X"
