File: Carte Alimentation/Batteries LiPo V1 (2015)/Carte Alim.kicad_pcb (KiCad board)
At the start: 2 copper layers, 102.9 x 70.5 mm, 58 parts, among them K1 CONN_01X03, P1 CONN_01X02, P10 CONN_01X02, P11 CONN_01X02, P12 CONN_01X02, P13 CONN_01X04, P2 CONN_01X02, P3 CONN_01X02, P4 CONN_01X05, P5 CONN_01X01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

Commit message: Réparation Alim 2015, remplacement du 7905 (régul -) par 7805 (régul +)
Parts:
- U100: value 7905_CORRIGE -> 7805
Changed lines of the file:
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@@
     (links 105)
     (no_connects 0)
-    (area 95.389999 76.404999 198.410001 147.040001)
+    (area 82.17 62.55 209.09 156.45)
     (thickness 1.6)
     (drawings 37)
@@
       (effects (font (size 1 1) (thickness 0.15)))
     )
-    (fp_text value 7905_CORRIGE (at 0 -3.1) (layer F.Fab)
+    (fp_text value 7805 (at 0 -3.1) (layer F.Fab)
       (effects (font (size 1 1) (thickness 0.15)))
     )
