File: Carte Alimentation/LiPo_module (2016)/LiPo_module.kicad_pcb (KiCad board)
At the start: 2 copper layers, 7 parts, among them P1 CONN_01X02, P2 CONN_01X02, P3 CONN_01X02, P4 CONN_01X02, U1 DSN2596, U2 DSN2596

Commit message: AJout condo céramiques aux sorties régulées (LiPo_module)
Parts:
- added C2: C, Capacitors_ThroughHole:C_Rect_L7_W2.5_P5, F.Cu at (171.4, 99.1)
- added C3: C, Capacitors_ThroughHole:C_Rect_L7_W2.5_P5, F.Cu at (171.4, 111.1)
Routing:
- net GND: track 180.4 -> 190.0 mm
