File: can-part.sch (KiCad schematic (older format))
At the start: 6 parts, among them P2 CAN bus, U5 MCP2562

Commit message: schematic seems ok, ongoing routing
Parts:
- P2: footprint Pin_Headers:Pin_Header_Straight_1x02 -> Connect:JWT_Vertical_A3963-RM3.96mm-2
Changed lines of the file:
@@
 $Descr A4 11693 8268
 encoding utf-8
-Sheet 4 7
+Sheet 4 9
 Title ""
 Date ""
@@
 	4050 3200 4200 3200
 $Comp
-L +5V #PWR036
+L +5V #PWR40
 U 1 1 5703AA77
 P 5100 2100
-F 0 "#PWR036" H 5100 1950 50  0001 C CNN
+F 0 "#PWR40" H 5100 1950 50  0001 C CNN
 F 1 "+5V" H 5118 2273 50  0000 C CNN
 F 2 "" H 5100 2100 50  0000 C CNN
@@
 $EndComp
 $Comp
-L GND #PWR037
+L GND #PWR41
 U 1 1 5703AB2D
 P 5400 2550
-F 0 "#PWR037" H 5400 2300 50  0001 C CNN
+F 0 "#PWR41" H 5400 2300 50  0001 C CNN
 F 1 "GND" H 5550 2450 50  0000 C CNN
 F 2 "" H 5400 2550 50  0000 C CNN
@@
 Connection ~ 4700 2250
 $Comp
-L GND #PWR038
+L GND #PWR37
 U 1 1 5703AC12
 P 4400 2550
-F 0 "#PWR038" H 4400 2300 50  0001 C CNN
+F 0 "#PWR37" H 4400 2300 50  0001 C CNN
 F 1 "GND" H 4300 2450 50  0000 C CNN
 F 2 "" H 4400 2550 50  0000 C CNN
@@
 	4400 2550 4400 2500
 $Comp
-L +3.3V #PWR039
+L +3.3V #PWR38
 U 1 1 5703AC64
 P 4700 2100
-F 0 "#PWR039" H 4700 1950 50  0001 C CNN
+F 0 "#PWR38" H 4700 1950 50  0001 C CNN
 F 1 "+3.3V" H 4718 2273 50  0000 C CNN
 F 2 "" H 4700 2100 50  0000 C CNN
@@
 F 0 "P2" H 6927 3238 50  0000 L CNN
 F 1 "CAN bus" H 6927 3147 50  0000 L CNN
-F 2 "Pin_Headers:Pin_Header_Straight_1x02" H 6850 3200 50  0001 C CNN
+F 2 "Connect:JWT_Vertical_A3963-RM3.96mm-2" H 6850 3200 50  0001 C CNN
 F 3 "" H 6850 3200 50  0000 C CNN
 	1    6850 3200
@@
 Connection ~ 5900 3500
 $Comp
-L GND #PWR040
+L GND #PWR39
 U 1 1 5703B0FD
 P 4900 3850
-F 0 "#PWR040" H 4900 3600 50  0001 C CNN
+F 0 "#PWR39" H 4900 3600 50  0001 C CNN
 F 1 "GND" H 4908 3677 50  0000 C CNN
 F 2 "" H 4900 3850 50  0000 C CNN
@@
 	5650 3000 5600 3000
 $Comp
-L GND #PWR041
+L GND #PWR36
 U 1 1 57053560
 P 4150 3450
-F 0 "#PWR041" H 4150 3200 50  0001 C CNN
+F 0 "#PWR36" H 4150 3200 50  0001 C CNN
 F 1 "GND" H 4158 3277 50  0000 C CNN
 F 2 "" H 4150 3450 50  0000 C CNN
