File: usb-part.sch (KiCad schematic (older format))
At the start: 8 parts, among them P3 USB_OTG, U7 USBLC6-2

Commit message: schematic seems ok, ongoing routing
Parts:
- C16: footprint Capacitors_SMD:C_1206 -> Capacitors_SMD:C_0805
- D5: value D_Small -> MBR0530T1G; footprint TO_SOT_Packages_SMD:SOT-23 -> Diodes_SMD:SOD-123
- P3: value USB_OTG -> usb
Changed lines of the file:
@@
 $Descr A4 11693 8268
 encoding utf-8
-Sheet 5 7
+Sheet 5 9
 Title ""
 Date ""
@@
 dp
 $Comp
-L GND #PWR042
+L GND #PWR48
 U 1 1 57018687
 P 4400 3350
-F 0 "#PWR042" H 4400 3100 50  0001 C CNN
+F 0 "#PWR48" H 4400 3100 50  0001 C CNN
 F 1 "GND" H 4408 3177 50  0000 C CNN
 F 2 "" H 4400 3350 50  0000 C CNN
@@
 P 4750 3050
 F 0 "P3" V 4777 3244 50  0000 L CNN
-F 1 "USB_OTG" V 4868 3244 50  0000 L CNN
+F 1 "usb" V 4868 3244 50  0000 L CNN
 F 2 "Connect:USB_Mini-B" V 4700 2950 50  0001 C CNN
 F 3 "" V 4700 2950 50  0000 C CNN
@@
 $EndComp
 $Comp
-L GND #PWR043
+L GND #PWR46
 U 1 1 57049AB6
 P 4200 3550
-F 0 "#PWR043" H 4200 3300 50  0001 C CNN
+F 0 "#PWR46" H 4200 3300 50  0001 C CNN
 F 1 "GND" H 4208 3377 50  0000 C CNN
 F 2 "" H 4200 3550 50  0000 C CNN
@@
 P 4300 2600
 F 0 "D5" V 4254 2668 50  0000 L CNN
-F 1 "D_Small" V 4345 2668 50  0000 L CNN
-F 2 "TO_SOT_Packages_SMD:SOT-23" V 4300 2600 50  0001 C CNN
+F 1 "MBR0530T1G" V 4345 2668 50  0000 L CNN
+F 2 "Diodes_SMD:SOD-123" V 4300 2600 50  0001 C CNN
 F 3 "" V 4300 2600 50  0000 C CNN
 	1    4300 2600
@@
 $EndComp
 $Comp
-L +5V #PWR044
+L +5V #PWR47
 U 1 1 5704AB79
 P 4300 2350
-F 0 "#PWR044" H 4300 2200 50  0001 C CNN
+F 0 "#PWR47" H 4300 2200 50  0001 C CNN
 F 1 "+5V" H 4318 2523 50  0000 C CNN
 F 2 "" H 4300 2350 50  0000 C CNN
@@
 $EndComp
 $Comp
-L GND #PWR045
+L GND #PWR44
 U 1 1 5704B58F
 P 2700 3400
-F 0 "#PWR045" H 2700 3150 50  0001 C CNN
+F 0 "#PWR44" H 2700 3150 50  0001 C CNN
 F 1 "GND" H 2708 3227 50  0000 C CNN
 F 2 "" H 2700 3400 50  0000 C CNN
@@
 F 0 "C16" V 2221 2500 50  0000 C CNN
 F 1 "100n" V 2312 2500 50  0000 C CNN
-F 2 "Capacitors_SMD:C_1206" H 2450 2500 50  0001 C CNN
+F 2 "Capacitors_SMD:C_0805" H 2450 2500 50  0001 C CNN
 F 3 "" H 2450 2500 50  0000 C CNN
 	1    2450 2500
@@
 $EndComp
 $Comp
-L GND #PWR046
+L GND #PWR42
 U 1 1 5704B7AF
 P 2350 2500
-F 0 "#PWR046" H 2350 2250 50  0001 C CNN
+F 0 "#PWR42" H 2350 2250 50  0001 C CNN
 F 1 "GND" H 2250 2400 50  0000 C CNN
 F 2 "" H 2350 2500 50  0000 C CNN
@@
 	2550 2500 2700 2500
 $Comp
-L +5V #PWR047
-U 1 1 5704B82A
-P 2700 2350
-F 0 "#PWR047" H 2700 2200 50  0001 C CNN
-F 1 "+5V" H 2718 2523 50  0000 C CNN
-F 2 "" H 2700 2350 50  0000 C CNN
-F 3 "" H 2700 2350 50  0000 C CNN
-	1    2700 2350
-	1    0    0    -1
-$EndComp
-$Comp
-L +3.3V #PWR048
+L +3.3V #PWR45
 U 1 1 57062CC0
 P 3900 2350
-F 0 "#PWR048" H 3900 2200 50  0001 C CNN
+F 0 "#PWR45" H 3900 2200 50  0001 C CNN
 F 1 "+3.3V" H 3918 2523 50  0000 C CNN
 F 2 "" H 3900 2350 50  0000 C CNN
@@
 Wire Wire Line
 	4200 3150 4200 3300
+$Comp
+L +5V #PWR43
+U 1 1 5704B82A
+P 2700 2350
+F 0 "#PWR43" H 2700 2200 50  0001 C CNN
+F 1 "+5V" H 2718 2523 50  0000 C CNN
+F 2 "" H 2700 2350 50  0000 C CNN
+F 3 "" H 2700 2350 50  0000 C CNN
+	1    2700 2350
+	1    0    0    -1
+$EndComp
 $EndSCHEMATC
