File: Sous-Carte Asservissement brushless EC-45-flat/can-part.sch (KiCad schematic (older format))
At the start: 6 parts, among them P2 CAN bus, U5 MCP2562

Commit message: added B-plugs for power
Parts:
- P2: footprint Connect:JWT_Vertical_A3963-RM3.96mm-2 -> Pin_Headers:Pin_Header_Straight_1x02
Changed lines of the file:
@@
 	4050 3200 4200 3200
 $Comp
-L +5V #PWR40
+L +5V #PWR035
 U 1 1 5703AA77
 P 5100 2100
-F 0 "#PWR40" H 5100 1950 50  0001 C CNN
+F 0 "#PWR035" H 5100 1950 50  0001 C CNN
 F 1 "+5V" H 5118 2273 50  0000 C CNN
 F 2 "" H 5100 2100 50  0000 C CNN
@@
 $EndComp
 $Comp
-L GND #PWR41
+L GND #PWR036
 U 1 1 5703AB2D
 P 5400 2550
-F 0 "#PWR41" H 5400 2300 50  0001 C CNN
+F 0 "#PWR036" H 5400 2300 50  0001 C CNN
 F 1 "GND" H 5550 2450 50  0000 C CNN
 F 2 "" H 5400 2550 50  0000 C CNN
@@
 Connection ~ 4700 2250
 $Comp
-L GND #PWR37
+L GND #PWR037
 U 1 1 5703AC12
 P 4400 2550
-F 0 "#PWR37" H 4400 2300 50  0001 C CNN
+F 0 "#PWR037" H 4400 2300 50  0001 C CNN
 F 1 "GND" H 4300 2450 50  0000 C CNN
 F 2 "" H 4400 2550 50  0000 C CNN
@@
 	4400 2550 4400 2500
 $Comp
-L +3.3V #PWR38
+L +3.3V #PWR038
 U 1 1 5703AC64
 P 4700 2100
-F 0 "#PWR38" H 4700 1950 50  0001 C CNN
+F 0 "#PWR038" H 4700 1950 50  0001 C CNN
 F 1 "+3.3V" H 4718 2273 50  0000 C CNN
 F 2 "" H 4700 2100 50  0000 C CNN
@@
 F 3 "" H 5900 3300 50  0000 C CNN
 	1    5900 3300
-	1    0    0    -1
-$EndComp
-$Comp
-L CONN_01X02 P2
-U 1 1 5703AD4C
-P 6850 3200
-F 0 "P2" H 6927 3238 50  0000 L CNN
-F 1 "CAN bus" H 6927 3147 50  0000 L CNN
-F 2 "Connect:JWT_Vertical_A3963-RM3.96mm-2" H 6850 3200 50  0001 C CNN
-F 3 "" H 6850 3200 50  0000 C CNN
-	1    6850 3200
 	1    0    0    -1
 $EndComp
@@
 Connection ~ 5900 3500
 $Comp
-L GND #PWR39
+L GND #PWR039
 U 1 1 5703B0FD
 P 4900 3850
-F 0 "#PWR39" H 4900 3600 50  0001 C CNN
+F 0 "#PWR039" H 4900 3600 50  0001 C CNN
 F 1 "GND" H 4908 3677 50  0000 C CNN
 F 2 "" H 4900 3850 50  0000 C CNN
@@
 	5650 3000 5600 3000
 $Comp
-L GND #PWR36
+L GND #PWR040
 U 1 1 57053560
 P 4150 3450
-F 0 "#PWR36" H 4150 3200 50  0001 C CNN
+F 0 "#PWR040" H 4150 3200 50  0001 C CNN
 F 1 "GND" H 4158 3277 50  0000 C CNN
 F 2 "" H 4150 3450 50  0000 C CNN
@@
 Wire Wire Line
 	4150 3400 4150 3450
+$Comp
+L CONN_01X02 P2
+U 1 1 570964CD
+P 6850 3200
+F 0 "P2" H 6927 3238 50  0000 L CNN
+F 1 "CAN bus" H 6927 3147 50  0000 L CNN
+F 2 "Pin_Headers:Pin_Header_Straight_1x02" H 6850 3200 50  0001 C CNN
+F 3 "" H 6850 3200 50  0000 C CNN
+	1    6850 3200
+	1    0    0    -1
+$EndComp
 $EndSCHEMATC

Commit message: asser 1A : BOM + ready for pisa !
Parts:
- U5: manf# (none) -> MCP2562-E/SN
Changed lines of the file:
@@
 F 2 "Housings_SOIC:SOIC-8_3.9x4.9mm_Pitch1.27mm" H 5150 3200 60  0001 C CNN
 F 3 "" H 5150 3200 60  0000 C CNN
+F 4 "MCP2562-E/SN" H 4900 3200 60  0001 C CNN "manf#"
 	1    4900 3200
 	1    0    0    -1
