File: Sous-Carte Asservissement brushless EC-45-flat/uC-part.sch (KiCad schematic (older format))
At the start: 19 parts, among them P1 swdio, Q1 BC807, Q2 BC807, U4 stm32f042k6tx

Commit message: added a nice logo :)
Connections:
- net pwm1_pos: now also U4.18 (PA8); no longer U4.19 (PA9)
- net pwm2_pos: now also U4.19 (PA9); no longer U4.18 (PA8)
Changed lines of the file:
@@
 pwm2
 Text Label 5300 3950 0    60   ~ 0
+pwm2_pos
+Text Label 5300 4050 0    60   ~ 0
 pwm1_pos
-Text Label 5300 4050 0    60   ~ 0
-pwm2_pos
 Wire Wire Line
 	4050 2950 4050 2900

Commit message: asser 1A : BOM + ready for pisa !
Parts:
- Q1, Q2: manf# (none) -> bc807
- U4: manf# (none) -> STM32F042K6T6
Changed lines of the file:
@@
 F 2 "Housings_QFP:LQFP-32_7x7mm_Pitch0.8mm" H 4050 3750 60  0001 C CNN
 F 3 "" H 4050 3750 60  0000 C CNN
+F 4 "STM32F042K6T6" H 4400 3800 60  0001 C CNN "manf#"
 	1    4400 3800
 	1    0    0    -1
@@
 F 2 "TO_SOT_Packages_SMD:SOT-23" H 3950 6050 50  0001 C CNN
 F 3 "" H 3750 5950 50  0000 C CNN
+F 4 "bc807" H 3750 5950 60  0001 C CNN "manf#"
 	1    3750 5950
 	1    0    0    1
@@
 F 2 "TO_SOT_Packages_SMD:SOT-23" H 5100 6050 50  0001 C CNN
 F 3 "" H 4900 5950 50  0000 C CNN
+F 4 "bc807" H 4900 5950 60  0001 C CNN "manf#"
 	1    4900 5950
 	1    0    0    1
