File: Sous-Carte Asservissement brushless EC-45-flat/usb-part.sch (KiCad schematic (older format))
At the start: 8 parts, among them P3 usb, U7 USBLC6-2

Commit message: asser 1A : BOM + ready for pisa !
Parts:
- D5: manf# (none) -> mbr0530T1G
- U7: manf# (none) -> USBLC6-2SC6Y
Changed lines of the file:
@@
 F 2 "Diodes_SMD:SOD-123" V 4300 2600 50  0001 C CNN
 F 3 "" V 4300 2600 50  0000 C CNN
+F 4 "mbr0530T1G" V 4300 2600 60  0001 C CNN "manf#"
 	1    4300 2600
 	0    1    1    0
@@
 F 2 "TO_SOT_Packages_SMD:SOT-23-6" H 2700 3000 60  0001 C CNN
 F 3 "" H 2700 3000 60  0000 C CNN
+F 4 "USBLC6-2SC6Y" H 2700 3000 60  0001 C CNN "manf#"
 	1    2700 3000
 	1    0    0    -1
