File: Carte OlINPiades/2017/Matrice/Carte OlINPiades 2017 - Matrice.kicad_pcb (KiCad board)
At the start: 2 copper layers, 258 parts

Commit message: Matrice Ol'INP 32*32 sch + routage
Parts:
- removed H1, H2: PinHeader, Pin_Headers:Pin_Header_Straight_1x16
- added D1000: LED, LEDs:LED_0805, F.Cu at (124.7, 225.6)
- added D1001: LED, LEDs:LED_0805, F.Cu at (130.3, 225.6)
- added D1002: LED, LEDs:LED_0805, F.Cu at (135.8, 225.6)
- added D1003: LED, LEDs:LED_0805, F.Cu at (141.4, 225.6)
- added D1004: LED, LEDs:LED_0805, F.Cu at (147.0, 225.6)
- added D1005: LED, LEDs:LED_0805, F.Cu at (152.6, 225.6)
- added D1006: LED, LEDs:LED_0805, F.Cu at (158.2, 225.6)
- added D1007: LED, LEDs:LED_0805, F.Cu at (163.8, 225.6)
- added D1008: LED, LEDs:LED_0805, F.Cu at (169.4, 225.6)
- added D1009: LED, LEDs:LED_0805, F.Cu at (175.0, 225.6)
- added D1010: LED, LEDs:LED_0805, F.Cu at (180.6, 225.6)
- added D1011: LED, LEDs:LED_0805, F.Cu at (186.1, 225.6)
- added D1012: LED, LEDs:LED_0805, F.Cu at (191.7, 225.6)
- added D1013: LED, LEDs:LED_0805, F.Cu at (197.3, 225.6)
- added D1014: LED, LEDs:LED_0805, F.Cu at (202.9, 225.6)
- added D1015: LED, LEDs:LED_0805, F.Cu at (208.5, 225.6)
- added D1016: LED, LEDs:LED_0805, F.Cu at (214.1, 225.6)
- added D1017: LED, LEDs:LED_0805, F.Cu at (219.7, 225.6)
- added D1018: LED, LEDs:LED_0805, F.Cu at (225.3, 225.6)
- added D1019: LED, LEDs:LED_0805, F.Cu at (230.8, 225.6)
- added D1020: LED, LEDs:LED_0805, F.Cu at (236.4, 225.6)
- added D1021: LED, LEDs:LED_0805, F.Cu at (242.0, 225.6)
- added D1022: LED, LEDs:LED_0805, F.Cu at (247.6, 225.6)
- added D1023: LED, LEDs:LED_0805, F.Cu at (253.2, 225.6)
- added D1024: LED, LEDs:LED_0805, F.Cu at (258.8, 225.6)
- added D257: LED, LEDs:LED_0805, F.Cu at (85.6, 97.1)
- added D258: LED, LEDs:LED_0805, F.Cu at (91.1, 97.1)
- added D259: LED, LEDs:LED_0805, F.Cu at (96.7, 97.1)
- added D260: LED, LEDs:LED_0805, F.Cu at (102.3, 97.1)
- added D261: LED, LEDs:LED_0805, F.Cu at (107.9, 97.1)
- added D262: LED, LEDs:LED_0805, F.Cu at (113.5, 97.1)
- added D263: LED, LEDs:LED_0805, F.Cu at (119.1, 97.1)
- added D264: LED, LEDs:LED_0805, F.Cu at (124.7, 97.1)
- added D265: LED, LEDs:LED_0805, F.Cu at (130.3, 97.1)
- added D266: LED, LEDs:LED_0805, F.Cu at (135.8, 97.1)
- added D267: LED, LEDs:LED_0805, F.Cu at (141.4, 97.1)
- added D268: LED, LEDs:LED_0805, F.Cu at (147.0, 97.1)
- added D269: LED, LEDs:LED_0805, F.Cu at (152.6, 97.1)
- added D270: LED, LEDs:LED_0805, F.Cu at (158.2, 97.1)
- added D271: LED, LEDs:LED_0805, F.Cu at (163.8, 97.1)
- added D272: LED, LEDs:LED_0805, F.Cu at (169.4, 97.1)
- added D273: LED, LEDs:LED_0805, F.Cu at (175.0, 97.1)
- added D274: LED, LEDs:LED_0805, F.Cu at (180.6, 97.1)
- added D275: LED, LEDs:LED_0805, F.Cu at (186.1, 97.1)
- added D276: LED, LEDs:LED_0805, F.Cu at (191.7, 97.1)
- added D277: LED, LEDs:LED_0805, F.Cu at (197.3, 97.1)
- added D278: LED, LEDs:LED_0805, F.Cu at (202.9, 97.1)
- added D279: LED, LEDs:LED_0805, F.Cu at (208.5, 97.1)
- added D280: LED, LEDs:LED_0805, F.Cu at (214.1, 97.1)
- added D281: LED, LEDs:LED_0805, F.Cu at (219.7, 97.1)
- added D282: LED, LEDs:LED_0805, F.Cu at (225.3, 97.1)
- added D283: LED, LEDs:LED_0805, F.Cu at (230.8, 97.1)
- added D284: LED, LEDs:LED_0805, F.Cu at (236.4, 97.1)
- added D285: LED, LEDs:LED_0805, F.Cu at (242.0, 97.1)
- added D286: LED, LEDs:LED_0805, F.Cu at (247.6, 97.1)
- added D287: LED, LEDs:LED_0805, F.Cu at (253.2, 97.1)
- added D288: LED, LEDs:LED_0805, F.Cu at (258.8, 97.1)
- added D289: LED, LEDs:LED_0805, F.Cu at (85.6, 102.6)
- added D290: LED, LEDs:LED_0805, F.Cu at (91.1, 102.6)
- added D291: LED, LEDs:LED_0805, F.Cu at (96.7, 102.6)
- added D292: LED, LEDs:LED_0805, F.Cu at (102.3, 102.6)
- added D293: LED, LEDs:LED_0805, F.Cu at (107.9, 102.6)
- added D294: LED, LEDs:LED_0805, F.Cu at (113.5, 102.6)
- added D295: LED, LEDs:LED_0805, F.Cu at (119.1, 102.6)
- added D296: LED, LEDs:LED_0805, F.Cu at (124.7, 102.6)
- added D297: LED, LEDs:LED_0805, F.Cu at (130.3, 102.6)
- added D298: LED, LEDs:LED_0805, F.Cu at (135.8, 102.6)
- added D299: LED, LEDs:LED_0805, F.Cu at (141.4, 102.6)
- added D300: LED, LEDs:LED_0805, F.Cu at (147.0, 102.6)
- added D301: LED, LEDs:LED_0805, F.Cu at (152.6, 102.6)
- added D302: LED, LEDs:LED_0805, F.Cu at (158.2, 102.6)
- added D303: LED, LEDs:LED_0805, F.Cu at (163.8, 102.6)
- added D304: LED, LEDs:LED_0805, F.Cu at (169.4, 102.6)
- added D305: LED, LEDs:LED_0805, F.Cu at (175.0, 102.6)
- added D306: LED, LEDs:LED_0805, F.Cu at (180.6, 102.6)
- added D307: LED, LEDs:LED_0805, F.Cu at (186.1, 102.6)
- added D308: LED, LEDs:LED_0805, F.Cu at (191.7, 102.6)
- added D309: LED, LEDs:LED_0805, F.Cu at (197.3, 102.6)
- added D310: LED, LEDs:LED_0805, F.Cu at (202.9, 102.6)
- added D311: LED, LEDs:LED_0805, F.Cu at (208.5, 102.6)
- added D312: LED, LEDs:LED_0805, F.Cu at (214.1, 102.6)
- added D313: LED, LEDs:LED_0805, F.Cu at (219.7, 102.6)
- added D314: LED, LEDs:LED_0805, F.Cu at (225.3, 102.6)
- added D315: LED, LEDs:LED_0805, F.Cu at (230.8, 102.6)
- added D316: LED, LEDs:LED_0805, F.Cu at (236.4, 102.6)
- added D317: LED, LEDs:LED_0805, F.Cu at (242.0, 102.6)
- added D318: LED, LEDs:LED_0805, F.Cu at (247.6, 102.6)
- added D319: LED, LEDs:LED_0805, F.Cu at (253.2, 102.6)
- added D320: LED, LEDs:LED_0805, F.Cu at (258.8, 102.6)
- added D321: LED, LEDs:LED_0805, F.Cu at (85.6, 108.2)
- added D322: LED, LEDs:LED_0805, F.Cu at (91.1, 108.2)
- added D323: LED, LEDs:LED_0805, F.Cu at (96.7, 108.2)
- added D324: LED, LEDs:LED_0805, F.Cu at (102.3, 108.2)
- added D325: LED, LEDs:LED_0805, F.Cu at (107.9, 108.2)
- added D326: LED, LEDs:LED_0805, F.Cu at (113.5, 108.2)
- added D327: LED, LEDs:LED_0805, F.Cu at (119.1, 108.2)
- added D328: LED, LEDs:LED_0805, F.Cu at (124.7, 108.2)
- added D329: LED, LEDs:LED_0805, F.Cu at (130.3, 108.2)
- added D330: LED, LEDs:LED_0805, F.Cu at (135.8, 108.2)
- added D331: LED, LEDs:LED_0805, F.Cu at (141.4, 108.2)
- added D332: LED, LEDs:LED_0805, F.Cu at (147.0, 108.2)
- added D333: LED, LEDs:LED_0805, F.Cu at (152.6, 108.2)
- added D334: LED, LEDs:LED_0805, F.Cu at (158.2, 108.2)
- added D335: LED, LEDs:LED_0805, F.Cu at (163.8, 108.2)
- added D336: LED, LEDs:LED_0805, F.Cu at (169.4, 108.2)
- added D337: LED, LEDs:LED_0805, F.Cu at (175.0, 108.2)
- added D338: LED, LEDs:LED_0805, F.Cu at (180.6, 108.2)
- added D339: LED, LEDs:LED_0805, F.Cu at (186.1, 108.2)
- added D340: LED, LEDs:LED_0805, F.Cu at (191.7, 108.2)
- added D341: LED, LEDs:LED_0805, F.Cu at (197.3, 108.2)
- added D342: LED, LEDs:LED_0805, F.Cu at (202.9, 108.2)
- added D343: LED, LEDs:LED_0805, F.Cu at (208.5, 108.2)
- added D344: LED, LEDs:LED_0805, F.Cu at (214.1, 108.2)
- added D345: LED, LEDs:LED_0805, F.Cu at (219.7, 108.2)
- added D346: LED, LEDs:LED_0805, F.Cu at (225.3, 108.2)
- added D347: LED, LEDs:LED_0805, F.Cu at (230.8, 108.2)
- added D348: LED, LEDs:LED_0805, F.Cu at (236.4, 108.2)
- added D349: LED, LEDs:LED_0805, F.Cu at (242.0, 108.2)
- added D350: LED, LEDs:LED_0805, F.Cu at (247.6, 108.2)
- added D351: LED, LEDs:LED_0805, F.Cu at (253.2, 108.2)
- added D352: LED, LEDs:LED_0805, F.Cu at (258.8, 108.2)
- added D353: LED, LEDs:LED_0805, F.Cu at (85.6, 113.8)
- added D354: LED, LEDs:LED_0805, F.Cu at (91.1, 113.8)
- added D355: LED, LEDs:LED_0805, F.Cu at (96.7, 113.8)
- added D356: LED, LEDs:LED_0805, F.Cu at (102.3, 113.8)
- added D357: LED, LEDs:LED_0805, F.Cu at (107.9, 113.8)
- added D358: LED, LEDs:LED_0805, F.Cu at (113.5, 113.8)
- added D359: LED, LEDs:LED_0805, F.Cu at (119.1, 113.8)
- added D360: LED, LEDs:LED_0805, F.Cu at (124.7, 113.8)
- added D361: LED, LEDs:LED_0805, F.Cu at (130.3, 113.8)
- added D362: LED, LEDs:LED_0805, F.Cu at (135.8, 113.8)
- added D363: LED, LEDs:LED_0805, F.Cu at (141.4, 113.8)
- added D364: LED, LEDs:LED_0805, F.Cu at (147.0, 113.8)
- added D365: LED, LEDs:LED_0805, F.Cu at (152.6, 113.8)
- added D366: LED, LEDs:LED_0805, F.Cu at (158.2, 113.8)
- added D367: LED, LEDs:LED_0805, F.Cu at (163.8, 113.8)
- added D368: LED, LEDs:LED_0805, F.Cu at (169.4, 113.8)
- added D369: LED, LEDs:LED_0805, F.Cu at (175.0, 113.8)
- added D370: LED, LEDs:LED_0805, F.Cu at (180.6, 113.8)
- added D371: LED, LEDs:LED_0805, F.Cu at (186.1, 113.8)
- added D372: LED, LEDs:LED_0805, F.Cu at (191.7, 113.8)
- added D373: LED, LEDs:LED_0805, F.Cu at (197.3, 113.8)
- added D374: LED, LEDs:LED_0805, F.Cu at (202.9, 113.8)
- added D375: LED, LEDs:LED_0805, F.Cu at (208.5, 113.8)
- added D376: LED, LEDs:LED_0805, F.Cu at (214.1, 113.8)
- added D377: LED, LEDs:LED_0805, F.Cu at (219.7, 113.8)
- added D378: LED, LEDs:LED_0805, F.Cu at (225.3, 113.8)
- added D379: LED, LEDs:LED_0805, F.Cu at (230.8, 113.8)
- added D380: LED, LEDs:LED_0805, F.Cu at (236.4, 113.8)
- added D381: LED, LEDs:LED_0805, F.Cu at (242.0, 113.8)
- added D382: LED, LEDs:LED_0805, F.Cu at (247.6, 113.8)
- added D383: LED, LEDs:LED_0805, F.Cu at (253.2, 113.8)
- added D384: LED, LEDs:LED_0805, F.Cu at (258.8, 113.8)
- added D385: LED, LEDs:LED_0805, F.Cu at (85.6, 119.4)
- added D386: LED, LEDs:LED_0805, F.Cu at (91.1, 119.4)
- added D387: LED, LEDs:LED_0805, F.Cu at (96.7, 119.4)
- added D388: LED, LEDs:LED_0805, F.Cu at (102.3, 119.4)
- added D389: LED, LEDs:LED_0805, F.Cu at (107.9, 119.4)
- added D390: LED, LEDs:LED_0805, F.Cu at (113.5, 119.4)
- added D391: LED, LEDs:LED_0805, F.Cu at (119.1, 119.4)
- added D392: LED, LEDs:LED_0805, F.Cu at (124.7, 119.4)
- added D393: LED, LEDs:LED_0805, F.Cu at (130.3, 119.4)
- added D394: LED, LEDs:LED_0805, F.Cu at (135.8, 119.4)
- added D395: LED, LEDs:LED_0805, F.Cu at (141.4, 119.4)
- added D396: LED, LEDs:LED_0805, F.Cu at (147.0, 119.4)
- added D397: LED, LEDs:LED_0805, F.Cu at (152.6, 119.4)
- added D398: LED, LEDs:LED_0805, F.Cu at (158.2, 119.4)
- added D399: LED, LEDs:LED_0805, F.Cu at (163.8, 119.4)
- added D400: LED, LEDs:LED_0805, F.Cu at (169.4, 119.4)
- added D401: LED, LEDs:LED_0805, F.Cu at (175.0, 119.4)
- added D402: LED, LEDs:LED_0805, F.Cu at (180.6, 119.4)
- added D403: LED, LEDs:LED_0805, F.Cu at (186.1, 119.4)
- added D404: LED, LEDs:LED_0805, F.Cu at (191.7, 119.4)
- added D405: LED, LEDs:LED_0805, F.Cu at (197.3, 119.4)
- added D406: LED, LEDs:LED_0805, F.Cu at (202.9, 119.4)
- added D407: LED, LEDs:LED_0805, F.Cu at (208.5, 119.4)
- added D408: LED, LEDs:LED_0805, F.Cu at (214.1, 119.4)
- added D409: LED, LEDs:LED_0805, F.Cu at (219.7, 119.4)
- added D410: LED, LEDs:LED_0805, F.Cu at (225.3, 119.4)
- added D411: LED, LEDs:LED_0805, F.Cu at (230.8, 119.4)
- added D412: LED, LEDs:LED_0805, F.Cu at (236.4, 119.4)
- added D413: LED, LEDs:LED_0805, F.Cu at (242.0, 119.4)
- added D414: LED, LEDs:LED_0805, F.Cu at (247.6, 119.4)
- added D415: LED, LEDs:LED_0805, F.Cu at (253.2, 119.4)
- added D416: LED, LEDs:LED_0805, F.Cu at (258.8, 119.4)
- added D417: LED, LEDs:LED_0805, F.Cu at (85.6, 125.0)
- added D418: LED, LEDs:LED_0805, F.Cu at (91.1, 125.0)
- added D419: LED, LEDs:LED_0805, F.Cu at (96.7, 125.0)
- added D420: LED, LEDs:LED_0805, F.Cu at (102.3, 125.0)
- added D421: LED, LEDs:LED_0805, F.Cu at (107.9, 125.0)
- added D422: LED, LEDs:LED_0805, F.Cu at (113.5, 125.0)
- added D423: LED, LEDs:LED_0805, F.Cu at (119.1, 125.0)
- added D424: LED, LEDs:LED_0805, F.Cu at (124.7, 125.0)
- added D425: LED, LEDs:LED_0805, F.Cu at (130.3, 125.0)
- added D426: LED, LEDs:LED_0805, F.Cu at (135.8, 125.0)
- added D427: LED, LEDs:LED_0805, F.Cu at (141.4, 125.0)
- added D428: LED, LEDs:LED_0805, F.Cu at (147.0, 125.0)
- added D429: LED, LEDs:LED_0805, F.Cu at (152.6, 125.0)
- added D430: LED, LEDs:LED_0805, F.Cu at (158.2, 125.0)
- added D431: LED, LEDs:LED_0805, F.Cu at (163.8, 125.0)
- added D432: LED, LEDs:LED_0805, F.Cu at (169.4, 125.0)
- added D433: LED, LEDs:LED_0805, F.Cu at (175.0, 125.0)
- added D434: LED, LEDs:LED_0805, F.Cu at (180.6, 125.0)
- added D435: LED, LEDs:LED_0805, F.Cu at (186.1, 125.0)
- added D436: LED, LEDs:LED_0805, F.Cu at (191.7, 125.0)
- added D437: LED, LEDs:LED_0805, F.Cu at (197.3, 125.0)
- added D438: LED, LEDs:LED_0805, F.Cu at (202.9, 125.0)
- added D439: LED, LEDs:LED_0805, F.Cu at (208.5, 125.0)
- added D440: LED, LEDs:LED_0805, F.Cu at (214.1, 125.0)
- added D441: LED, LEDs:LED_0805, F.Cu at (219.7, 125.0)
- added D442: LED, LEDs:LED_0805, F.Cu at (225.3, 125.0)
- added D443: LED, LEDs:LED_0805, F.Cu at (230.8, 125.0)
- added D444: LED, LEDs:LED_0805, F.Cu at (236.4, 125.0)
- added D445: LED, LEDs:LED_0805, F.Cu at (242.0, 125.0)
- added D446: LED, LEDs:LED_0805, F.Cu at (247.6, 125.0)
- added D447: LED, LEDs:LED_0805, F.Cu at (253.2, 125.0)
- added D448: LED, LEDs:LED_0805, F.Cu at (258.8, 125.0)
- added D449: LED, LEDs:LED_0805, F.Cu at (85.6, 130.6)
- added D450: LED, LEDs:LED_0805, F.Cu at (91.1, 130.6)
- added D451: LED, LEDs:LED_0805, F.Cu at (96.7, 130.6)
- added D452: LED, LEDs:LED_0805, F.Cu at (102.3, 130.6)
- added D453: LED, LEDs:LED_0805, F.Cu at (107.9, 130.6)
- added D454: LED, LEDs:LED_0805, F.Cu at (113.5, 130.6)
- added D455: LED, LEDs:LED_0805, F.Cu at (119.1, 130.6)
- added D456: LED, LEDs:LED_0805, F.Cu at (124.7, 130.6)
- added D457: LED, LEDs:LED_0805, F.Cu at (130.3, 130.6)
- added D458: LED, LEDs:LED_0805, F.Cu at (135.8, 130.6)
- added D459: LED, LEDs:LED_0805, F.Cu at (141.4, 130.6)
- added D460: LED, LEDs:LED_0805, F.Cu at (147.0, 130.6)
- added D461: LED, LEDs:LED_0805, F.Cu at (152.6, 130.6)
- added D462: LED, LEDs:LED_0805, F.Cu at (158.2, 130.6)
- added D463: LED, LEDs:LED_0805, F.Cu at (163.8, 130.6)
- added D464: LED, LEDs:LED_0805, F.Cu at (169.4, 130.6)
- added D465: LED, LEDs:LED_0805, F.Cu at (175.0, 130.6)
- added D466: LED, LEDs:LED_0805, F.Cu at (180.6, 130.6)
- added D467: LED, LEDs:LED_0805, F.Cu at (186.1, 130.6)
- added D468: LED, LEDs:LED_0805, F.Cu at (191.7, 130.6)
- added D469: LED, LEDs:LED_0805, F.Cu at (197.3, 130.6)
- added D470: LED, LEDs:LED_0805, F.Cu at (202.9, 130.6)
- added D471: LED, LEDs:LED_0805, F.Cu at (208.5, 130.6)
- added D472: LED, LEDs:LED_0805, F.Cu at (214.1, 130.6)
- added D473: LED, LEDs:LED_0805, F.Cu at (219.7, 130.6)
- added D474: LED, LEDs:LED_0805, F.Cu at (225.3, 130.6)
- added D475: LED, LEDs:LED_0805, F.Cu at (230.8, 130.6)
- added D476: LED, LEDs:LED_0805, F.Cu at (236.4, 130.6)
- added D477: LED, LEDs:LED_0805, F.Cu at (242.0, 130.6)
- added D478: LED, LEDs:LED_0805, F.Cu at (247.6, 130.6)
- added D479: LED, LEDs:LED_0805, F.Cu at (253.2, 130.6)
- added D480: LED, LEDs:LED_0805, F.Cu at (258.8, 130.6)
- added D481: LED, LEDs:LED_0805, F.Cu at (85.6, 136.2)
- added D482: LED, LEDs:LED_0805, F.Cu at (91.1, 136.2)
- added D483: LED, LEDs:LED_0805, F.Cu at (96.7, 136.2)
- added D484: LED, LEDs:LED_0805, F.Cu at (102.3, 136.2)
- added D485: LED, LEDs:LED_0805, F.Cu at (107.9, 136.2)
- added D486: LED, LEDs:LED_0805, F.Cu at (113.5, 136.2)
- added D487: LED, LEDs:LED_0805, F.Cu at (119.1, 136.2)
- added D488: LED, LEDs:LED_0805, F.Cu at (124.7, 136.2)
- added D489: LED, LEDs:LED_0805, F.Cu at (130.3, 136.2)
- added D490: LED, LEDs:LED_0805, F.Cu at (135.8, 136.2)
- added D491: LED, LEDs:LED_0805, F.Cu at (141.4, 136.2)
- added D492: LED, LEDs:LED_0805, F.Cu at (147.0, 136.2)
- added D493: LED, LEDs:LED_0805, F.Cu at (152.6, 136.2)
- added D494: LED, LEDs:LED_0805, F.Cu at (158.2, 136.2)
- added D495: LED, LEDs:LED_0805, F.Cu at (163.8, 136.2)
- added D496: LED, LEDs:LED_0805, F.Cu at (169.4, 136.2)
- added D497: LED, LEDs:LED_0805, F.Cu at (175.0, 136.2)
- added D498: LED, LEDs:LED_0805, F.Cu at (180.6, 136.2)
- added D499: LED, LEDs:LED_0805, F.Cu at (186.1, 136.2)
- added D500: LED, LEDs:LED_0805, F.Cu at (191.7, 136.2)
- added D501: LED, LEDs:LED_0805, F.Cu at (197.3, 136.2)
- added D502: LED, LEDs:LED_0805, F.Cu at (202.9, 136.2)
- added D503: LED, LEDs:LED_0805, F.Cu at (208.5, 136.2)
- added D504: LED, LEDs:LED_0805, F.Cu at (214.1, 136.2)
- added D505: LED, LEDs:LED_0805, F.Cu at (219.7, 136.2)
- added D506: LED, LEDs:LED_0805, F.Cu at (225.3, 136.2)
- added D507: LED, LEDs:LED_0805, F.Cu at (230.8, 136.2)
- added D508: LED, LEDs:LED_0805, F.Cu at (236.4, 136.2)
- added D509: LED, LEDs:LED_0805, F.Cu at (242.0, 136.2)
- added D510: LED, LEDs:LED_0805, F.Cu at (247.6, 136.2)
- added D511: LED, LEDs:LED_0805, F.Cu at (253.2, 136.2)
- added D512: LED, LEDs:LED_0805, F.Cu at (258.8, 136.2)
- added D513: LED, LEDs:LED_0805, F.Cu at (85.6, 141.8)
- added D514: LED, LEDs:LED_0805, F.Cu at (91.1, 141.8)
- added D515: LED, LEDs:LED_0805, F.Cu at (96.7, 141.8)
- added D516: LED, LEDs:LED_0805, F.Cu at (102.3, 141.8)
- added D517: LED, LEDs:LED_0805, F.Cu at (107.9, 141.8)
- added D518: LED, LEDs:LED_0805, F.Cu at (113.5, 141.8)
- added D519: LED, LEDs:LED_0805, F.Cu at (119.1, 141.8)
- added D520: LED, LEDs:LED_0805, F.Cu at (124.7, 141.8)
- added D521: LED, LEDs:LED_0805, F.Cu at (130.3, 141.8)
- added D522: LED, LEDs:LED_0805, F.Cu at (135.8, 141.8)
- added D523: LED, LEDs:LED_0805, F.Cu at (141.4, 141.8)
- added D524: LED, LEDs:LED_0805, F.Cu at (147.0, 141.8)
- added D525: LED, LEDs:LED_0805, F.Cu at (152.6, 141.8)
- added D526: LED, LEDs:LED_0805, F.Cu at (158.2, 141.8)
- added D527: LED, LEDs:LED_0805, F.Cu at (163.8, 141.8)
- added D528: LED, LEDs:LED_0805, F.Cu at (169.4, 141.8)
- added D529: LED, LEDs:LED_0805, F.Cu at (175.0, 141.8)
- added D530: LED, LEDs:LED_0805, F.Cu at (180.6, 141.8)
- added D531: LED, LEDs:LED_0805, F.Cu at (186.1, 141.8)
- added D532: LED, LEDs:LED_0805, F.Cu at (191.7, 141.8)
- added D533: LED, LEDs:LED_0805, F.Cu at (197.3, 141.8)
- added D534: LED, LEDs:LED_0805, F.Cu at (202.9, 141.8)
- added D535: LED, LEDs:LED_0805, F.Cu at (208.5, 141.8)
- added D536: LED, LEDs:LED_0805, F.Cu at (214.1, 141.8)
- added D537: LED, LEDs:LED_0805, F.Cu at (219.7, 141.8)
- added D538: LED, LEDs:LED_0805, F.Cu at (225.3, 141.8)
- added D539: LED, LEDs:LED_0805, F.Cu at (230.8, 141.8)
- added D540: LED, LEDs:LED_0805, F.Cu at (236.4, 141.8)
- added D541: LED, LEDs:LED_0805, F.Cu at (242.0, 141.8)
- added D542: LED, LEDs:LED_0805, F.Cu at (247.6, 141.8)
- added D543: LED, LEDs:LED_0805, F.Cu at (253.2, 141.8)
- added D544: LED, LEDs:LED_0805, F.Cu at (258.8, 141.8)
- added D545: LED, LEDs:LED_0805, F.Cu at (85.6, 147.3)
- added D546: LED, LEDs:LED_0805, F.Cu at (91.1, 147.3)
- added D547: LED, LEDs:LED_0805, F.Cu at (96.7, 147.3)
- added D548: LED, LEDs:LED_0805, F.Cu at (102.3, 147.3)
- added D549: LED, LEDs:LED_0805, F.Cu at (107.9, 147.3)
- added D550: LED, LEDs:LED_0805, F.Cu at (113.5, 147.3)
- added D551: LED, LEDs:LED_0805, F.Cu at (119.1, 147.3)
- added D552: LED, LEDs:LED_0805, F.Cu at (124.7, 147.3)
- added D553: LED, LEDs:LED_0805, F.Cu at (130.3, 147.3)
- added D554: LED, LEDs:LED_0805, F.Cu at (135.8, 147.3)
- added D555: LED, LEDs:LED_0805, F.Cu at (141.4, 147.3)
- added D556: LED, LEDs:LED_0805, F.Cu at (147.0, 147.3)
- added D557: LED, LEDs:LED_0805, F.Cu at (152.6, 147.3)
- added D558: LED, LEDs:LED_0805, F.Cu at (158.2, 147.3)
- added D559: LED, LEDs:LED_0805, F.Cu at (163.8, 147.3)
- added D560: LED, LEDs:LED_0805, F.Cu at (169.4, 147.3)
- added D561: LED, LEDs:LED_0805, F.Cu at (175.0, 147.3)
- added D562: LED, LEDs:LED_0805, F.Cu at (180.6, 147.3)
- added D563: LED, LEDs:LED_0805, F.Cu at (186.1, 147.3)
- added D564: LED, LEDs:LED_0805, F.Cu at (191.7, 147.3)
- added D565: LED, LEDs:LED_0805, F.Cu at (197.3, 147.3)
- added D566: LED, LEDs:LED_0805, F.Cu at (202.9, 147.3)
- added D567: LED, LEDs:LED_0805, F.Cu at (208.5, 147.3)
- added D568: LED, LEDs:LED_0805, F.Cu at (214.1, 147.3)
- added D569: LED, LEDs:LED_0805, F.Cu at (219.7, 147.3)
- added D570: LED, LEDs:LED_0805, F.Cu at (225.3, 147.3)
- added D571: LED, LEDs:LED_0805, F.Cu at (230.8, 147.3)
- added D572: LED, LEDs:LED_0805, F.Cu at (236.4, 147.3)
- added D573: LED, LEDs:LED_0805, F.Cu at (242.0, 147.3)
- added D574: LED, LEDs:LED_0805, F.Cu at (247.6, 147.3)
- added D575: LED, LEDs:LED_0805, F.Cu at (253.2, 147.3)
- added D576: LED, LEDs:LED_0805, F.Cu at (258.8, 147.3)
- added D577: LED, LEDs:LED_0805, F.Cu at (85.6, 152.9)
- added D578: LED, LEDs:LED_0805, F.Cu at (91.1, 152.9)
- added D579: LED, LEDs:LED_0805, F.Cu at (96.7, 152.9)
- added D580: LED, LEDs:LED_0805, F.Cu at (102.3, 152.9)
- added D581: LED, LEDs:LED_0805, F.Cu at (107.9, 152.9)
- added D582: LED, LEDs:LED_0805, F.Cu at (113.5, 152.9)
- added D583: LED, LEDs:LED_0805, F.Cu at (119.1, 152.9)
- added D584: LED, LEDs:LED_0805, F.Cu at (124.7, 152.9)
- added D585: LED, LEDs:LED_0805, F.Cu at (130.3, 152.9)
- added D586: LED, LEDs:LED_0805, F.Cu at (135.8, 152.9)
- added D587: LED, LEDs:LED_0805, F.Cu at (141.4, 152.9)
- added D588: LED, LEDs:LED_0805, F.Cu at (147.0, 152.9)
- added D589: LED, LEDs:LED_0805, F.Cu at (152.6, 152.9)
- added D590: LED, LEDs:LED_0805, F.Cu at (158.2, 152.9)
- added D591: LED, LEDs:LED_0805, F.Cu at (163.8, 152.9)
- added D592: LED, LEDs:LED_0805, F.Cu at (169.4, 152.9)
- added D593: LED, LEDs:LED_0805, F.Cu at (175.0, 152.9)
- added D594: LED, LEDs:LED_0805, F.Cu at (180.6, 152.9)
- added D595: LED, LEDs:LED_0805, F.Cu at (186.1, 152.9)
- added D596: LED, LEDs:LED_0805, F.Cu at (191.7, 152.9)
- added D597: LED, LEDs:LED_0805, F.Cu at (197.3, 152.9)
- added D598: LED, LEDs:LED_0805, F.Cu at (202.9, 152.9)
- added D599: LED, LEDs:LED_0805, F.Cu at (208.5, 152.9)
- added D600: LED, LEDs:LED_0805, F.Cu at (214.1, 152.9)
- added D601: LED, LEDs:LED_0805, F.Cu at (219.7, 152.9)
- added D602: LED, LEDs:LED_0805, F.Cu at (225.3, 152.9)
- added D603: LED, LEDs:LED_0805, F.Cu at (230.8, 152.9)
- added D604: LED, LEDs:LED_0805, F.Cu at (236.4, 152.9)
- added D605: LED, LEDs:LED_0805, F.Cu at (242.0, 152.9)
- added D606: LED, LEDs:LED_0805, F.Cu at (247.6, 152.9)
- added D607: LED, LEDs:LED_0805, F.Cu at (253.2, 152.9)
- added D608: LED, LEDs:LED_0805, F.Cu at (258.8, 152.9)
- added D609: LED, LEDs:LED_0805, F.Cu at (85.6, 158.5)
- added D610: LED, LEDs:LED_0805, F.Cu at (91.1, 158.5)
- added D611: LED, LEDs:LED_0805, F.Cu at (96.7, 158.5)
- added D612: LED, LEDs:LED_0805, F.Cu at (102.3, 158.5)
- added D613: LED, LEDs:LED_0805, F.Cu at (107.9, 158.5)
- added D614: LED, LEDs:LED_0805, F.Cu at (113.5, 158.5)
- added D615: LED, LEDs:LED_0805, F.Cu at (119.1, 158.5)
- added D616: LED, LEDs:LED_0805, F.Cu at (124.7, 158.5)
- added D617: LED, LEDs:LED_0805, F.Cu at (130.3, 158.5)
- added D618: LED, LEDs:LED_0805, F.Cu at (135.8, 158.5)
- added D619: LED, LEDs:LED_0805, F.Cu at (141.4, 158.5)
- added D620: LED, LEDs:LED_0805, F.Cu at (147.0, 158.5)
- added D621: LED, LEDs:LED_0805, F.Cu at (152.6, 158.5)
- added D622: LED, LEDs:LED_0805, F.Cu at (158.2, 158.5)
- added D623: LED, LEDs:LED_0805, F.Cu at (163.8, 158.5)
- added D624: LED, LEDs:LED_0805, F.Cu at (169.4, 158.5)
- added D625: LED, LEDs:LED_0805, F.Cu at (175.0, 158.5)
- added D626: LED, LEDs:LED_0805, F.Cu at (180.6, 158.5)
- added D627: LED, LEDs:LED_0805, F.Cu at (186.1, 158.5)
- added D628: LED, LEDs:LED_0805, F.Cu at (191.7, 158.5)
- added D629: LED, LEDs:LED_0805, F.Cu at (197.3, 158.5)
- added D630: LED, LEDs:LED_0805, F.Cu at (202.9, 158.5)
- added D631: LED, LEDs:LED_0805, F.Cu at (208.5, 158.5)
- added D632: LED, LEDs:LED_0805, F.Cu at (214.1, 158.5)
- added D633: LED, LEDs:LED_0805, F.Cu at (219.7, 158.5)
- added D634: LED, LEDs:LED_0805, F.Cu at (225.3, 158.5)
- added D635: LED, LEDs:LED_0805, F.Cu at (230.8, 158.5)
- added D636: LED, LEDs:LED_0805, F.Cu at (236.4, 158.5)
- added D637: LED, LEDs:LED_0805, F.Cu at (242.0, 158.5)
- added D638: LED, LEDs:LED_0805, F.Cu at (247.6, 158.5)
- added D639: LED, LEDs:LED_0805, F.Cu at (253.2, 158.5)
- added D640: LED, LEDs:LED_0805, F.Cu at (258.8, 158.5)
- added D641: LED, LEDs:LED_0805, F.Cu at (85.6, 164.1)
- added D642: LED, LEDs:LED_0805, F.Cu at (91.1, 164.1)
- added D643: LED, LEDs:LED_0805, F.Cu at (96.7, 164.1)
- added D644: LED, LEDs:LED_0805, F.Cu at (102.3, 164.1)
- added D645: LED, LEDs:LED_0805, F.Cu at (107.9, 164.1)
- added D646: LED, LEDs:LED_0805, F.Cu at (113.5, 164.1)
- added D647: LED, LEDs:LED_0805, F.Cu at (119.1, 164.1)
- added D648: LED, LEDs:LED_0805, F.Cu at (124.7, 164.1)
- added D649: LED, LEDs:LED_0805, F.Cu at (130.3, 164.1)
- added D650: LED, LEDs:LED_0805, F.Cu at (135.8, 164.1)
- added D651: LED, LEDs:LED_0805, F.Cu at (141.4, 164.1)
- added D652: LED, LEDs:LED_0805, F.Cu at (147.0, 164.1)
- added D653: LED, LEDs:LED_0805, F.Cu at (152.6, 164.1)
- added D654: LED, LEDs:LED_0805, F.Cu at (158.2, 164.1)
- added D655: LED, LEDs:LED_0805, F.Cu at (163.8, 164.1)
- added D656: LED, LEDs:LED_0805, F.Cu at (169.4, 164.1)
- added D657: LED, LEDs:LED_0805, F.Cu at (175.0, 164.1)
- added D658: LED, LEDs:LED_0805, F.Cu at (180.6, 164.1)
- added D659: LED, LEDs:LED_0805, F.Cu at (186.1, 164.1)
- added D660: LED, LEDs:LED_0805, F.Cu at (191.7, 164.1)
- added D661: LED, LEDs:LED_0805, F.Cu at (197.3, 164.1)
- added D662: LED, LEDs:LED_0805, F.Cu at (202.9, 164.1)
- added D663: LED, LEDs:LED_0805, F.Cu at (208.5, 164.1)
- added D664: LED, LEDs:LED_0805, F.Cu at (214.1, 164.1)
- added D665: LED, LEDs:LED_0805, F.Cu at (219.7, 164.1)
- added D666: LED, LEDs:LED_0805, F.Cu at (225.3, 164.1)
- added D667: LED, LEDs:LED_0805, F.Cu at (230.8, 164.1)
- added D668: LED, LEDs:LED_0805, F.Cu at (236.4, 164.1)
- added D669: LED, LEDs:LED_0805, F.Cu at (242.0, 164.1)
- added D670: LED, LEDs:LED_0805, F.Cu at (247.6, 164.1)
- added D671: LED, LEDs:LED_0805, F.Cu at (253.2, 164.1)
- added D672: LED, LEDs:LED_0805, F.Cu at (258.8, 164.1)
- added D673: LED, LEDs:LED_0805, F.Cu at (85.6, 169.7)
- added D674: LED, LEDs:LED_0805, F.Cu at (91.1, 169.7)
- added D675: LED, LEDs:LED_0805, F.Cu at (96.7, 169.7)
- added D676: LED, LEDs:LED_0805, F.Cu at (102.3, 169.7)
- added D677: LED, LEDs:LED_0805, F.Cu at (107.9, 169.7)
- added D678: LED, LEDs:LED_0805, F.Cu at (113.5, 169.7)
- added D679: LED, LEDs:LED_0805, F.Cu at (119.1, 169.7)
- added D680: LED, LEDs:LED_0805, F.Cu at (124.7, 169.7)
- added D681: LED, LEDs:LED_0805, F.Cu at (130.3, 169.7)
- added D682: LED, LEDs:LED_0805, F.Cu at (135.8, 169.7)
- added D683: LED, LEDs:LED_0805, F.Cu at (141.4, 169.7)
- added D684: LED, LEDs:LED_0805, F.Cu at (147.0, 169.7)
- added D685: LED, LEDs:LED_0805, F.Cu at (152.6, 169.7)
- added D686: LED, LEDs:LED_0805, F.Cu at (158.2, 169.7)
- added D687: LED, LEDs:LED_0805, F.Cu at (163.8, 169.7)
- added D688: LED, LEDs:LED_0805, F.Cu at (169.4, 169.7)
- added D689: LED, LEDs:LED_0805, F.Cu at (175.0, 169.7)
- added D690: LED, LEDs:LED_0805, F.Cu at (180.6, 169.7)
- added D691: LED, LEDs:LED_0805, F.Cu at (186.1, 169.7)
- added D692: LED, LEDs:LED_0805, F.Cu at (191.7, 169.7)
- added D693: LED, LEDs:LED_0805, F.Cu at (197.3, 169.7)
- added D694: LED, LEDs:LED_0805, F.Cu at (202.9, 169.7)
- added D695: LED, LEDs:LED_0805, F.Cu at (208.5, 169.7)
- added D696: LED, LEDs:LED_0805, F.Cu at (214.1, 169.7)
- added D697: LED, LEDs:LED_0805, F.Cu at (219.7, 169.7)
- added D698: LED, LEDs:LED_0805, F.Cu at (225.3, 169.7)
- added D699: LED, LEDs:LED_0805, F.Cu at (230.8, 169.7)
- added D700: LED, LEDs:LED_0805, F.Cu at (236.4, 169.7)
- added D701: LED, LEDs:LED_0805, F.Cu at (242.0, 169.7)
- added D702: LED, LEDs:LED_0805, F.Cu at (247.6, 169.7)
- added D703: LED, LEDs:LED_0805, F.Cu at (253.2, 169.7)
- added D704: LED, LEDs:LED_0805, F.Cu at (258.8, 169.7)
- added D705: LED, LEDs:LED_0805, F.Cu at (85.6, 175.3)
- added D706: LED, LEDs:LED_0805, F.Cu at (91.1, 175.3)
- added D707: LED, LEDs:LED_0805, F.Cu at (96.7, 175.3)
- added D708: LED, LEDs:LED_0805, F.Cu at (102.3, 175.3)
- added D709: LED, LEDs:LED_0805, F.Cu at (107.9, 175.3)
- added D710: LED, LEDs:LED_0805, F.Cu at (113.5, 175.3)
- added D711: LED, LEDs:LED_0805, F.Cu at (119.1, 175.3)
- added D712: LED, LEDs:LED_0805, F.Cu at (124.7, 175.3)
- added D713: LED, LEDs:LED_0805, F.Cu at (130.3, 175.3)
- added D714: LED, LEDs:LED_0805, F.Cu at (135.8, 175.3)
- added D715: LED, LEDs:LED_0805, F.Cu at (141.4, 175.3)
- added D716: LED, LEDs:LED_0805, F.Cu at (147.0, 175.3)
- added D717: LED, LEDs:LED_0805, F.Cu at (152.6, 175.3)
- added D718: LED, LEDs:LED_0805, F.Cu at (158.2, 175.3)
- added D719: LED, LEDs:LED_0805, F.Cu at (163.8, 175.3)
- added D720: LED, LEDs:LED_0805, F.Cu at (169.4, 175.3)
- added D721: LED, LEDs:LED_0805, F.Cu at (175.0, 175.3)
- added D722: LED, LEDs:LED_0805, F.Cu at (180.6, 175.3)
- added D723: LED, LEDs:LED_0805, F.Cu at (186.1, 175.3)
- added D724: LED, LEDs:LED_0805, F.Cu at (191.7, 175.3)
- added D725: LED, LEDs:LED_0805, F.Cu at (197.3, 175.3)
- added D726: LED, LEDs:LED_0805, F.Cu at (202.9, 175.3)
- added D727: LED, LEDs:LED_0805, F.Cu at (208.5, 175.3)
- added D728: LED, LEDs:LED_0805, F.Cu at (214.1, 175.3)
- added D729: LED, LEDs:LED_0805, F.Cu at (219.7, 175.3)
- added D730: LED, LEDs:LED_0805, F.Cu at (225.3, 175.3)
- added D731: LED, LEDs:LED_0805, F.Cu at (230.8, 175.3)
- added D732: LED, LEDs:LED_0805, F.Cu at (236.4, 175.3)
- added D733: LED, LEDs:LED_0805, F.Cu at (242.0, 175.3)
- added D734: LED, LEDs:LED_0805, F.Cu at (247.6, 175.3)
- added D735: LED, LEDs:LED_0805, F.Cu at (253.2, 175.3)
- added D736: LED, LEDs:LED_0805, F.Cu at (258.8, 175.3)
- added D737: LED, LEDs:LED_0805, F.Cu at (85.6, 180.9)
- added D738: LED, LEDs:LED_0805, F.Cu at (91.1, 180.9)
- added D739: LED, LEDs:LED_0805, F.Cu at (96.7, 180.9)
- added D740: LED, LEDs:LED_0805, F.Cu at (102.3, 180.9)
- added D741: LED, LEDs:LED_0805, F.Cu at (107.9, 180.9)
- added D742: LED, LEDs:LED_0805, F.Cu at (113.5, 180.9)
- added D743: LED, LEDs:LED_0805, F.Cu at (119.1, 180.9)
- added D744: LED, LEDs:LED_0805, F.Cu at (124.7, 180.9)
- added D745: LED, LEDs:LED_0805, F.Cu at (130.3, 180.9)
- added D746: LED, LEDs:LED_0805, F.Cu at (135.8, 180.9)
- added D747: LED, LEDs:LED_0805, F.Cu at (141.4, 180.9)
- added D748: LED, LEDs:LED_0805, F.Cu at (147.0, 180.9)
- added D749: LED, LEDs:LED_0805, F.Cu at (152.6, 180.9)
- added D750: LED, LEDs:LED_0805, F.Cu at (158.2, 180.9)
- added D751: LED, LEDs:LED_0805, F.Cu at (163.8, 180.9)
- added D752: LED, LEDs:LED_0805, F.Cu at (169.4, 180.9)
- added D753: LED, LEDs:LED_0805, F.Cu at (175.0, 180.9)
- added D754: LED, LEDs:LED_0805, F.Cu at (180.6, 180.9)
- added D755: LED, LEDs:LED_0805, F.Cu at (186.1, 180.9)
- added D756: LED, LEDs:LED_0805, F.Cu at (191.7, 180.9)
- added D757: LED, LEDs:LED_0805, F.Cu at (197.3, 180.9)
- added D758: LED, LEDs:LED_0805, F.Cu at (202.9, 180.9)
- added D759: LED, LEDs:LED_0805, F.Cu at (208.5, 180.9)
- added D760: LED, LEDs:LED_0805, F.Cu at (214.1, 180.9)
- added D761: LED, LEDs:LED_0805, F.Cu at (219.7, 180.9)
- added D762: LED, LEDs:LED_0805, F.Cu at (225.3, 180.9)
- added D763: LED, LEDs:LED_0805, F.Cu at (230.8, 180.9)
- added D764: LED, LEDs:LED_0805, F.Cu at (236.4, 180.9)
- added D765: LED, LEDs:LED_0805, F.Cu at (242.0, 180.9)
- added D766: LED, LEDs:LED_0805, F.Cu at (247.6, 180.9)
- added D767: LED, LEDs:LED_0805, F.Cu at (253.2, 180.9)
- added D768: LED, LEDs:LED_0805, F.Cu at (258.8, 180.9)
- added D769: LED, LEDs:LED_0805, F.Cu at (85.6, 186.5)
- added D770: LED, LEDs:LED_0805, F.Cu at (91.1, 186.5)
- added D771: LED, LEDs:LED_0805, F.Cu at (96.7, 186.5)
- added D772: LED, LEDs:LED_0805, F.Cu at (102.3, 186.5)
- added D773: LED, LEDs:LED_0805, F.Cu at (107.9, 186.5)
- added D774: LED, LEDs:LED_0805, F.Cu at (113.5, 186.5)
- added D775: LED, LEDs:LED_0805, F.Cu at (119.1, 186.5)
- added D776: LED, LEDs:LED_0805, F.Cu at (124.7, 186.5)
- added D777: LED, LEDs:LED_0805, F.Cu at (130.3, 186.5)
- added D778: LED, LEDs:LED_0805, F.Cu at (135.8, 186.5)
- added D779: LED, LEDs:LED_0805, F.Cu at (141.4, 186.5)
- added D780: LED, LEDs:LED_0805, F.Cu at (147.0, 186.5)
- added D781: LED, LEDs:LED_0805, F.Cu at (152.6, 186.5)
- added D782: LED, LEDs:LED_0805, F.Cu at (158.2, 186.5)
- added D783: LED, LEDs:LED_0805, F.Cu at (163.8, 186.5)
- added D784: LED, LEDs:LED_0805, F.Cu at (169.4, 186.5)
- added D785: LED, LEDs:LED_0805, F.Cu at (175.0, 186.5)
- added D786: LED, LEDs:LED_0805, F.Cu at (180.6, 186.5)
- added D787: LED, LEDs:LED_0805, F.Cu at (186.1, 186.5)
- added D788: LED, LEDs:LED_0805, F.Cu at (191.7, 186.5)
- added D789: LED, LEDs:LED_0805, F.Cu at (197.3, 186.5)
- added D790: LED, LEDs:LED_0805, F.Cu at (202.9, 186.5)
- added D791: LED, LEDs:LED_0805, F.Cu at (208.5, 186.5)
- added D792: LED, LEDs:LED_0805, F.Cu at (214.1, 186.5)
- added D793: LED, LEDs:LED_0805, F.Cu at (219.7, 186.5)
- added D794: LED, LEDs:LED_0805, F.Cu at (225.3, 186.5)
- added D795: LED, LEDs:LED_0805, F.Cu at (230.8, 186.5)
- added D796: LED, LEDs:LED_0805, F.Cu at (236.4, 186.5)
- added D797: LED, LEDs:LED_0805, F.Cu at (242.0, 186.5)
- added D798: LED, LEDs:LED_0805, F.Cu at (247.6, 186.5)
- added D799: LED, LEDs:LED_0805, F.Cu at (253.2, 186.5)
- added D800: LED, LEDs:LED_0805, F.Cu at (258.8, 186.5)
- added D801: LED, LEDs:LED_0805, F.Cu at (85.6, 192.1)
- added D802: LED, LEDs:LED_0805, F.Cu at (91.1, 192.1)
- added D803: LED, LEDs:LED_0805, F.Cu at (96.7, 192.1)
- added D804: LED, LEDs:LED_0805, F.Cu at (102.3, 192.1)
- added D805: LED, LEDs:LED_0805, F.Cu at (107.9, 192.1)
- added D806: LED, LEDs:LED_0805, F.Cu at (113.5, 192.1)
- added D807: LED, LEDs:LED_0805, F.Cu at (119.1, 192.1)
- added D808: LED, LEDs:LED_0805, F.Cu at (124.7, 192.1)
- added D809: LED, LEDs:LED_0805, F.Cu at (130.3, 192.1)
- added D810: LED, LEDs:LED_0805, F.Cu at (135.8, 192.1)
- added D811: LED, LEDs:LED_0805, F.Cu at (141.4, 192.1)
- added D812: LED, LEDs:LED_0805, F.Cu at (147.0, 192.1)
- added D813: LED, LEDs:LED_0805, F.Cu at (152.6, 192.1)
- added D814: LED, LEDs:LED_0805, F.Cu at (158.2, 192.1)
- added D815: LED, LEDs:LED_0805, F.Cu at (163.8, 192.1)
- added D816: LED, LEDs:LED_0805, F.Cu at (169.4, 192.1)
- added D817: LED, LEDs:LED_0805, F.Cu at (175.0, 192.1)
- added D818: LED, LEDs:LED_0805, F.Cu at (180.6, 192.1)
- added D819: LED, LEDs:LED_0805, F.Cu at (186.1, 192.1)
- added D820: LED, LEDs:LED_0805, F.Cu at (191.7, 192.1)
- added D821: LED, LEDs:LED_0805, F.Cu at (197.3, 192.1)
- added D822: LED, LEDs:LED_0805, F.Cu at (202.9, 192.1)
- added D823: LED, LEDs:LED_0805, F.Cu at (208.5, 192.1)
- added D824: LED, LEDs:LED_0805, F.Cu at (214.1, 192.1)
- added D825: LED, LEDs:LED_0805, F.Cu at (219.7, 192.1)
- added D826: LED, LEDs:LED_0805, F.Cu at (225.3, 192.1)
- added D827: LED, LEDs:LED_0805, F.Cu at (230.8, 192.1)
- added D828: LED, LEDs:LED_0805, F.Cu at (236.4, 192.1)
- added D829: LED, LEDs:LED_0805, F.Cu at (242.0, 192.1)
- added D830: LED, LEDs:LED_0805, F.Cu at (247.6, 192.1)
- added D831: LED, LEDs:LED_0805, F.Cu at (253.2, 192.1)
- added D832: LED, LEDs:LED_0805, F.Cu at (258.8, 192.1)
- added D833: LED, LEDs:LED_0805, F.Cu at (85.6, 197.6)
- added D834: LED, LEDs:LED_0805, F.Cu at (91.1, 197.6)
- added D835: LED, LEDs:LED_0805, F.Cu at (96.7, 197.6)
- added D836: LED, LEDs:LED_0805, F.Cu at (102.3, 197.6)
- added D837: LED, LEDs:LED_0805, F.Cu at (107.9, 197.6)
- added D838: LED, LEDs:LED_0805, F.Cu at (113.5, 197.6)
- added D839: LED, LEDs:LED_0805, F.Cu at (119.1, 197.6)
- added D840: LED, LEDs:LED_0805, F.Cu at (124.7, 197.6)
- added D841: LED, LEDs:LED_0805, F.Cu at (130.3, 197.6)
- added D842: LED, LEDs:LED_0805, F.Cu at (135.8, 197.6)
- added D843: LED, LEDs:LED_0805, F.Cu at (141.4, 197.6)
- added D844: LED, LEDs:LED_0805, F.Cu at (147.0, 197.6)
- added D845: LED, LEDs:LED_0805, F.Cu at (152.6, 197.6)
- added D846: LED, LEDs:LED_0805, F.Cu at (158.2, 197.6)
- added D847: LED, LEDs:LED_0805, F.Cu at (163.8, 197.6)
- added D848: LED, LEDs:LED_0805, F.Cu at (169.4, 197.6)
- added D849: LED, LEDs:LED_0805, F.Cu at (175.0, 197.6)
- added D850: LED, LEDs:LED_0805, F.Cu at (180.6, 197.6)
- added D851: LED, LEDs:LED_0805, F.Cu at (186.1, 197.6)
- added D852: LED, LEDs:LED_0805, F.Cu at (191.7, 197.6)
- added D853: LED, LEDs:LED_0805, F.Cu at (197.3, 197.6)
- added D854: LED, LEDs:LED_0805, F.Cu at (202.9, 197.6)
- added D855: LED, LEDs:LED_0805, F.Cu at (208.5, 197.6)
- added D856: LED, LEDs:LED_0805, F.Cu at (214.1, 197.6)
- added D857: LED, LEDs:LED_0805, F.Cu at (219.7, 197.6)
- added D858: LED, LEDs:LED_0805, F.Cu at (225.3, 197.6)
- added D859: LED, LEDs:LED_0805, F.Cu at (230.8, 197.6)
- added D860: LED, LEDs:LED_0805, F.Cu at (236.4, 197.6)
- added D861: LED, LEDs:LED_0805, F.Cu at (242.0, 197.6)
- added D862: LED, LEDs:LED_0805, F.Cu at (247.6, 197.6)
- added D863: LED, LEDs:LED_0805, F.Cu at (253.2, 197.6)
- added D864: LED, LEDs:LED_0805, F.Cu at (258.8, 197.6)
- added D865: LED, LEDs:LED_0805, F.Cu at (85.6, 203.2)
- added D866: LED, LEDs:LED_0805, F.Cu at (91.1, 203.2)
- added D867: LED, LEDs:LED_0805, F.Cu at (96.7, 203.2)
- added D868: LED, LEDs:LED_0805, F.Cu at (102.3, 203.2)
- added D869: LED, LEDs:LED_0805, F.Cu at (107.9, 203.2)
- added D870: LED, LEDs:LED_0805, F.Cu at (113.5, 203.2)
- added D871: LED, LEDs:LED_0805, F.Cu at (119.1, 203.2)
- added D872: LED, LEDs:LED_0805, F.Cu at (124.7, 203.2)
- added D873: LED, LEDs:LED_0805, F.Cu at (130.3, 203.2)
- added D874: LED, LEDs:LED_0805, F.Cu at (135.8, 203.2)
- added D875: LED, LEDs:LED_0805, F.Cu at (141.4, 203.2)
- added D876: LED, LEDs:LED_0805, F.Cu at (147.0, 203.2)
- added D877: LED, LEDs:LED_0805, F.Cu at (152.6, 203.2)
- added D878: LED, LEDs:LED_0805, F.Cu at (158.2, 203.2)
- added D879: LED, LEDs:LED_0805, F.Cu at (163.8, 203.2)
- added D880: LED, LEDs:LED_0805, F.Cu at (169.4, 203.2)
- added D881: LED, LEDs:LED_0805, F.Cu at (175.0, 203.2)
- added D882: LED, LEDs:LED_0805, F.Cu at (180.6, 203.2)
- added D883: LED, LEDs:LED_0805, F.Cu at (186.1, 203.2)
- added D884: LED, LEDs:LED_0805, F.Cu at (191.7, 203.2)
- added D885: LED, LEDs:LED_0805, F.Cu at (197.3, 203.2)
- added D886: LED, LEDs:LED_0805, F.Cu at (202.9, 203.2)
- added D887: LED, LEDs:LED_0805, F.Cu at (208.5, 203.2)
- added D888: LED, LEDs:LED_0805, F.Cu at (214.1, 203.2)
- added D889: LED, LEDs:LED_0805, F.Cu at (219.7, 203.2)
- added D890: LED, LEDs:LED_0805, F.Cu at (225.3, 203.2)
- added D891: LED, LEDs:LED_0805, F.Cu at (230.8, 203.2)
- added D892: LED, LEDs:LED_0805, F.Cu at (236.4, 203.2)
- added D893: LED, LEDs:LED_0805, F.Cu at (242.0, 203.2)
- added D894: LED, LEDs:LED_0805, F.Cu at (247.6, 203.2)
- added D895: LED, LEDs:LED_0805, F.Cu at (253.2, 203.2)
- added D896: LED, LEDs:LED_0805, F.Cu at (258.8, 203.2)
- added D897: LED, LEDs:LED_0805, F.Cu at (85.6, 208.8)
- added D898: LED, LEDs:LED_0805, F.Cu at (91.1, 208.8)
- added D899: LED, LEDs:LED_0805, F.Cu at (96.7, 208.8)
- added D900: LED, LEDs:LED_0805, F.Cu at (102.3, 208.8)
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Connections:
- D10 pad 1: Net-(D1-Pad1) -> Net-(D10-Pad1)
- D10 pad 2: Net-(D10-Pad2) -> Net-(D1-Pad2)
- D101 pad 1: Net-(D100-Pad1) -> Net-(D101-Pad1)
- D101 pad 2: Net-(D101-Pad2) -> Net-(D100-Pad2)
- D102 pad 1: Net-(D100-Pad1) -> Net-(D102-Pad1)
- D102 pad 2: Net-(D102-Pad2) -> Net-(D100-Pad2)
- D103 pad 1: Net-(D100-Pad1) -> Net-(D103-Pad1)
- D103 pad 2: Net-(D103-Pad2) -> Net-(D100-Pad2)
- D104 pad 1: Net-(D100-Pad1) -> Net-(D1000-Pad1)
- D104 pad 2: Net-(D104-Pad2) -> Net-(D100-Pad2)
- D105 pad 1: Net-(D100-Pad1) -> Net-(D1001-Pad1)
- D105 pad 2: Net-(D105-Pad2) -> Net-(D100-Pad2)
- D106 pad 1: Net-(D100-Pad1) -> Net-(D10-Pad1)
- D106 pad 2: Net-(D10-Pad2) -> Net-(D100-Pad2)
- D107 pad 1: Net-(D100-Pad1) -> Net-(D1003-Pad1)
- D107 pad 2: Net-(D107-Pad2) -> Net-(D100-Pad2)
- D108 pad 1: Net-(D100-Pad1) -> Net-(D1004-Pad1)
- D108 pad 2: Net-(D108-Pad2) -> Net-(D100-Pad2)
- D109 pad 1: Net-(D100-Pad1) -> Net-(D1005-Pad1)
- D109 pad 2: Net-(D109-Pad2) -> Net-(D100-Pad2)
- D11 pad 1: Net-(D1-Pad1) -> Net-(D1003-Pad1)
- D11 pad 2: Net-(D107-Pad2) -> Net-(D1-Pad2)
- D110 pad 1: Net-(D100-Pad1) -> Net-(D1006-Pad1)
- D110 pad 2: Net-(D110-Pad2) -> Net-(D100-Pad2)
- D111 pad 1: Net-(D100-Pad1) -> Net-(D1007-Pad1)
- D111 pad 2: Net-(D111-Pad2) -> Net-(D100-Pad2)
- D112 pad 1: Net-(D100-Pad1) -> Net-(D1008-Pad1)
- D112 pad 2: Net-(D112-Pad2) -> Net-(D100-Pad2)
- D113 pad 1: Net-(D113-Pad1) -> Net-(D1009-Pad1)
- D113 pad 2: Net-(D1-Pad2) -> Net-(D100-Pad2)
- D114 pad 1: Net-(D113-Pad1) -> Net-(D1010-Pad1)
- D114 pad 2: Net-(D114-Pad2) -> Net-(D100-Pad2)
- D115 pad 1: Net-(D113-Pad1) -> Net-(D1011-Pad1)
- D115 pad 2: Net-(D115-Pad2) -> Net-(D100-Pad2)
- D116 pad 1: Net-(D113-Pad1) -> Net-(D1012-Pad1)
- D117 pad 1: Net-(D113-Pad1) -> Net-(D1013-Pad1)
- D117 pad 2: Net-(D101-Pad2) -> Net-(D100-Pad2)
- D118 pad 1: Net-(D113-Pad1) -> Net-(D1014-Pad1)
- D118 pad 2: Net-(D102-Pad2) -> Net-(D100-Pad2)
- D119 pad 1: Net-(D113-Pad1) -> Net-(D1015-Pad1)
- D119 pad 2: Net-(D103-Pad2) -> Net-(D100-Pad2)
- D12 pad 1: Net-(D1-Pad1) -> Net-(D1004-Pad1)
- D12 pad 2: Net-(D108-Pad2) -> Net-(D1-Pad2)
- D120 pad 1: Net-(D113-Pad1) -> Net-(D1016-Pad1)
- D120 pad 2: Net-(D104-Pad2) -> Net-(D100-Pad2)
- D121 pad 1: Net-(D113-Pad1) -> Net-(D1017-Pad1)
- D121 pad 2: Net-(D105-Pad2) -> Net-(D100-Pad2)
- D122 pad 1: Net-(D113-Pad1) -> Net-(D1018-Pad1)
- D122 pad 2: Net-(D10-Pad2) -> Net-(D100-Pad2)
- D123 pad 1: Net-(D113-Pad1) -> Net-(D1019-Pad1)
- D123 pad 2: Net-(D107-Pad2) -> Net-(D100-Pad2)
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Routing:
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Other:
- board outline added: 200 x 200 mm
- net class Seedstudio added: clearance 0.1524, trace_width 0.381, via_dia 0.762, via_drill 0.508

Commit message: Finalisation matrice
Parts:
- added G***: LOGO, drawings:robotronik_logo_big, B.Cu at (167.5, 138.5)
Other:
- board text added: "Matrice Ol'INP 2017"
