File: Carte-OlINPiades/2017/Logique/Carte OlINPiades 2017 - Logique.kicad_pcb (KiCad board)
At the start: 2 copper layers, 100 x 100 mm, 85 parts, among them P1 CONN_01X32, P2 CONN_01X32, P3 CONN_01X02, P4 CONN_01X05, P5 CONN_01X02, P6 CONN_01X02, Q1 MMPQ2907A, Q2 MMPQ2907A, Q3 MMPQ2907A, Q4 MMPQ2907A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

Commit message: modif empreinte STM32
Parts:
- removed the G*** at (167.0, 104.6)
- added C6: C, Capacitors_SMD:C_1206_HandSoldering, B.Cu at (180.3, 120.3)
- added C9: C, Capacitors_SMD:C_1206_HandSoldering, B.Cu at (173.2, 121.1)
- added JP1: JUMPER3, Pin_Headers:Pin_Header_Straight_1x03_Pitch2.54mm, F.Cu at (168.3, 85.7)
- added JP2: JUMPER, Resistors_SMD:R_1206_HandSoldering, F.Cu at (178.2, 112.9)
- added P7: CONN_FREE_01X03, Pin_Headers:Pin_Header_Straight_1x03_Pitch2.54mm, F.Cu at (191.7, 119.2)
- added R37: R, Resistors_SMD:R_1206_HandSoldering, B.Cu at (177.2, 114.1)
- added R38: 10kR, Resistors_SMD:R_1206_HandSoldering, F.Cu at (168.3, 94.1)
- added Y1: Crystal, Crystals:Crystal_HC49-4H_Vertical, F.Cu at (172.3, 118.7)
- C3: moved to F.Cu
- P4: value CONN_01X05 -> CONN_01X06; footprint Pin_Headers:Pin_Header_Angled_1x05 -> Pin_Headers:Pin_Header_Angled_1x06_Pitch2.54mm
- U4: footprint Housings_QFP:LQFP-32_5x5mm_Pitch0.5mm -> Housings_QFP:LQFP-32_7x7mm_Pitch0.8mm
- moved P6 7.54 mm to (171.7, 125.5)
- moved C3 6.76 mm to (172.3, 107.2), turned to 180 degrees
- moved U4 2.90 mm to (172.5, 105.5)
- moved P3 2.38 mm to (169.4, 138.8)
Connections:
- P4 pad 1: SWCLK -> GND
- P4 pad 2: SWDIO -> SWCLK
- P4 pad 3: NRST -> SWDIO
- P4 pad 4: JTDO -> NRST
- P4 pad 5: JTDI -> JTDO
- S2 pad 22: (no net) -> Net-(S2-Pad22)
- U1 pad 1: (no net) -> Net-(U1-Pad1)
- U4 pad 18: TX_SERIAL -> SERIAL_IN
- U4 pad 19: RX_SERIAL -> TX_SERIAL
- U4 pad 2: (no net) -> Net-(C9-Pad1)
- U4 pad 20: SERIAL_IN -> RX_SERIAL
- U4 pad 27: NRST -> Net-(JP2-Pad2)
- U4 pad 28: (no net) -> F3
- U4 pad 29: (no net) -> F2
- U4 pad 3: (no net) -> Net-(R37-Pad1)
- U4 pad 30: (no net) -> F1
- U4 pad 31: GND -> Net-(R38-Pad2)
- U5 pad 5: (no net) -> Net-(U5-Pad5)
Routing:
- net GND: track 284.7 -> 334.8 mm, vias 16 -> 15
- net F1: track 0.00 -> 20.1 mm, vias 0 -> 1
- net F2: track 0.00 -> 19.4 mm, vias 0 -> 1
- net F3: track 0.00 -> 18.7 mm, vias 0 -> 1
- net Net-(R38-Pad2): track 0.00 -> 16.1 mm, vias 0 -> 1
- net Net-(C9-Pad1): track 0.00 -> 13.6 mm, vias 0 -> 2
- net NRST: track 26.6 -> 38.5 mm, vias 3 -> 1
- net Net-(JP2-Pad2): track 0.00 -> 11.1 mm, vias 0 -> 1
- net TX_EYE: track 13.7 -> 23.5 mm
- net RX_EYE: track 12.4 -> 21.8 mm, vias 1 -> 2
- net Net-(JP1-Pad2): track 0.00 -> 7.46 mm
- net RX_SERIAL: track 38.2 -> 32.0 mm
- net TX_SERIAL: track 36.8 -> 30.7 mm
- net SWCLK: track 24.3 -> 18.4 mm, vias 0 -> 1
- net Net-(R37-Pad1): track 0.00 -> 5.07 mm
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